File: Hotp4ck60.kicad_pcb (KiCad board)
At the start: 2 copper layers, 285 x 96.2 mm, 196 parts, among them J1 HRO_TYPE-C-31-M-12, J3 Conn_01x02_MountingPin, Q1 2N7002, SW1 RST, SW2 PWR, U1 nRF52840, U2 SRV05-4, U3 BQ24075, U4 MAX17048, Y1 32 MHz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

Commit message: replace parts and change pin assignment.
Parts:
- moved D53 16.7 mm to (323.1, 155.6)
- moved D32 15.9 mm to (144.5, 136.5)
- moved D63 12.7 mm to (246.9, 165.1), turned to -90 degrees
- moved R12 9.92 mm to (168.9, 160.6), turned to 180 degrees
- moved R13 8.53 mm to (168.9, 161.6), turned to 180 degrees
- moved C18 0.88 mm to (164.0, 169.1), turned to -90 degrees
- moved C16 0.38 mm to (173.3, 166.7)
- moved C17 0.30 mm to (173.2, 169.9)
- moved C5 0.21 mm to (162.5, 169.6)
- moved C10 0.21 mm to (163.2, 165.5)
- moved C9 0.20 mm to (161.9, 164.9)
- moved F1 0.17 mm to (88.3, 96.8)
- moved L2 0.13 mm to (162.9, 163.2)
- moved R2 0.13 mm to (92.9, 94.6)
- moved R5 0.11 mm to (173.3, 167.8)
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Connections:
- S47 pad 1: col6 -> col5
- S48 pad 1: col7 -> col6
- S49 pad 1: col8 -> col7
- S50 pad 1: col9 -> col8
- S53 pad 1: col12 -> col13
- S63 pad 1: col6 -> col7
- U1 pad A12: unconnected-(U1-AIN0/P0.02-PadA12) -> col0
- U1 pad A14: col2 -> col1
- U1 pad A16: col1 -> col2
- U1 pad A20: col0 -> col3
- U1 pad AD10: SCL -> unconnected-(U1-P0.15-PadAD10)
- U1 pad AD8: SDA -> unconnected-(U1-P0.13-PadAD8)
- U1 pad G1: row3 -> unconnected-(U1-P0.26-PadG1)
- U1 pad J1: col3 -> unconnected-(U1-AIN2/P0.04-PadJ1)
- U1 pad L1: row2 -> unconnected-(U1-P0.06-PadL1)
- U1 pad N1: row0 -> unconnected-(U1-P0.08-PadN1)
- U1 pad R1: row1 -> SDA
- U1 pad U1: row4 -> SCL
Routing:
- net row1: track 6.14 -> 274.9 mm, vias 0 -> 2
- net row2: track 6.39 -> 232.8 mm, vias 0 -> 2
- net row0: track 6.09 -> 222.9 mm
- net row4: track 40.3 -> 255.2 mm, vias 1 -> 2
- net row3: track 7.77 -> 222.3 mm, vias 0 -> 2
- net col0: track 7.90 -> 177.0 mm
- net col1: track 7.71 -> 168.7 mm
- net col2: track 7.87 -> 131.4 mm
- net col5: track 0.17 -> 104.1 mm
- net col3: track 6.60 -> 104.4 mm
- net col13: track 13.5 -> 108.4 mm
- net col11: track 13.9 -> 101.0 mm
- net col10: track 13.5 -> 100.5 mm
- net col7: track 12.7 -> 99.7 mm
- net col12: track 13.0 -> 94.1 mm
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
Commit message: Routing finished
Parts:
- SW1: moved to B.Cu
- moved SW1 95.2 mm to (188.2, 164.3), turned to 180 degrees
- moved J2 90.5 mm to (178.2, 168.9), turned to 90 degrees
- moved LED1 48.1 mm to (104.1, 136.7)
- moved LED2 46.0 mm to (104.1, 134.5)
- moved J3 24.9 mm to (121.3, 124.9)
- moved R10 21.2 mm to (95.6, 124.2)
- moved R9 21.2 mm to (95.1, 122.7)
- moved R7 21.2 mm to (100.1, 124.2)
- moved C21 21.2 mm to (97.4, 128.6)
- moved C22 21.2 mm to (98.4, 128.6)
- moved C23 21.2 mm to (101.9, 130.1)
- moved C24 21.2 mm to (101.9, 131.1)
- moved C25 21.2 mm to (101.9, 123.5)
- moved C26 21.2 mm to (101.9, 124.5)
- moved Q1 21.2 mm to (97.9, 123.2)
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Connections:
- U1 pad A10: unconnected-(U1-AIN5/P0.29-PadA10) -> LED
- U1 pad AD10: unconnected-(U1-P0.15-PadAD10) -> row1
- U1 pad AD12: unconnected-(U1-P0.17-PadAD12) -> row2
- U1 pad AD16: LED -> col4
- U1 pad AD18: col4 -> row3
- U1 pad AD20: col5 -> col6
- U1 pad AD22: col6 -> col7
- U1 pad AD8: unconnected-(U1-P0.13-PadAD8) -> row0
- U1 pad N1: unconnected-(U1-P0.08-PadN1) -> row4
- U1 pad P23: col11 -> col10
- U1 pad T23: col10 -> col9
- U1 pad W24: col9 -> col11
- U1 pad Y23: col7 -> col5
Routing:
- net col13: track 108.4 -> 274.5 mm
- net col12: track 94.1 -> 239.2 mm
- net col9: track 56.6 -> 179.8 mm, vias 0 -> 1
- net col11: track 101.0 -> 220.8 mm, vias 1 -> 0
- net +5V: track 52.1 -> 170.5 mm, vias 0 -> 1
- net USB-D+: track 45.6 -> 152.4 mm, vias 2 -> 0
- net USB-D-: track 44.8 -> 151.2 mm, vias 2 -> 0
- net col10: track 100.5 -> 196.5 mm
- net col8: track 80.1 -> 175.4 mm
- net VDDH: track 32.1 -> 125.8 mm, vias 3 -> 6
- net SCL: track 8.54 -> 90.9 mm, vias 0 -> 2
- net SDA: track 9.00 -> 89.1 mm, vias 0 -> 2
- net row0: track 222.9 -> 302.7 mm, vias 0 -> 1
- net row1: track 274.9 -> 334.7 mm, vias 2 -> 4
- net col7: track 99.7 -> 158.6 mm
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- added copper zone on B.Cu, net GND
- added copper zone on F.Cu, net GND
- added copper zone on B.Cu, net GNDPWR
- added copper zone on F.Cu, net GNDPWR
Other:
- board text added: "On|Off"
- board text added: ""
- board text added: ""

Commit message: Enter LCSC parts numbers
Parts:
- moved R1 1.41 mm to (88.0, 95.7)
- moved L5 1.40 mm to (90.0, 95.7)
- moved F1 1.11 mm to (88.3, 97.9)
- moved J1 1.11 mm to (90.0, 89.5)
- moved R2 1.11 mm to (92.9, 95.7)
- moved U2 1.11 mm to (91.2, 98.1)
Connections:
- H8 pad 1: GND -> Earth
- J1 pad A1: GNDPWR -> GND
- J1 pad A12: GNDPWR -> GND
- J1 pad B1: GNDPWR -> GND
- J1 pad B12: GNDPWR -> GND
- J1 pad S1: GNDPWR -> Earth
- R1 pad 2: GNDPWR -> GND
- R2 pad 2: GNDPWR -> GND
- U1 pad J1: unconnected-(U1-AIN2/P0.04-PadJ1) -> row4
- U1 pad N1: row4 -> SDA
- U1 pad R1: SDA -> SCL
- U1 pad U1: SCL -> unconnected-(U1-TRACEDATA1/P0.12-PadU1)
Routing:
- net Earth: track 0.00 -> 45.6 mm
- net GNDPWR: track 15.1 -> 0.00 mm, vias 2 -> 0
- net GND: track 27.7 -> 41.1 mm
- net Net-(D1-A): track 28.9 -> 27.5 mm
- net +5V: track 170.5 -> 169.4 mm
- net Net-(F1-Pad1): track 1.52 -> 2.07 mm
- net Net-(J1-CC1): track 2.68 -> 2.18 mm
- removed copper zone on B.Cu, net GNDPWR
- removed copper zone on F.Cu, net GNDPWR
Other:
- board size 285 x 96.2 mm -> 285 x 94.6 mm

Commit message: Fixed position & etc..
Parts:
- added C28: 100nF, Capacitor_SMD:C_0402_1005Metric, B.Cu at (92.8, 96.7)
- added D64: D_TVS, Diode_SMD:D_SOD-123F, B.Cu at (93.8, 100.3)
- added L6: BLM15PX121SN1D, Inductor_SMD:L_0402_1005Metric, B.Cu at (91.3, 96.2)
- added R14: 1 MOhm, Resistor_SMD:R_0402_1005Metric, B.Cu at (92.8, 95.7)
- LED1: value blue -> Blue; footprint LED_SMD:LED_0402_1005Metric -> LED_SMD:LED_0603_1608Metric
- LED2: value orange -> Yellow; footprint LED_SMD:LED_0402_1005Metric -> LED_SMD:LED_0603_1608Metric
- moved R2 12.8 mm to (80.4, 93.0), turned to -90 degrees
- moved R1 7.16 mm to (81.4, 93.0), turned to -90 degrees
- moved D2 3.55 mm to (108.0, 98.4)
- moved D1 3.53 mm to (111.1, 98.4)
- moved L5 2.01 mm to (88.0, 96.0), turned to -90 degrees
- moved U2 1.93 mm to (90.5, 99.8)
- moved F1 1.70 mm to (89.3, 96.5)
- moved LED2 0.70 mm to (103.9, 133.8)
- moved LED1 0.38 mm to (103.9, 137.1)
Connections:
- J1 pad A1: GND -> GNDPWR
- J1 pad A12: GND -> GNDPWR
- J1 pad B1: GND -> GNDPWR
- J1 pad B12: GND -> GNDPWR
- R1 pad 2: GND -> GNDPWR
- R2 pad 2: GND -> GNDPWR
- U2 pad 1: unconnected-(U2-IO1-Pad1) -> USB-D-
- U2 pad 3: USB-D- -> unconnected-(U2-IO2-Pad3)
- U2 pad 4: USB-D+ -> unconnected-(U2-IO3-Pad4)
- U2 pad 6: unconnected-(U2-IO4-Pad6) -> USB-D+
Routing:
- net GNDPWR: track 0.00 -> 22.7 mm, vias 0 -> 2
- net Net-(J1-CC2): track 2.31 -> 15.8 mm, vias 0 -> 2
- net Earth: track 45.6 -> 55.4 mm
- net Net-(J1-CC1): track 2.18 -> 11.6 mm, vias 0 -> 2
- net GND: track 41.1 -> 32.2 mm, vias 362 -> 344
- net Net-(D1-A): track 27.5 -> 32.1 mm
- net +5V: track 169.4 -> 171.9 mm
- net USB-D-: track 151.3 -> 150.1 mm
- net Net-(D2-A): track 10.2 -> 9.28 mm
- net Net-(LED2-K): track 4.05 -> 3.13 mm
- net USB-D+: track 152.2 -> 151.4 mm
- net row0: track 302.7 -> 302.1 mm
- net Net-(LED1-A): track 76.7 -> 76.1 mm
- net VBUS: track 8.47 -> 8.26 mm, vias 3 -> 2
- added copper zone on B.Cu, net Earth
- added copper zone on F.Cu, net Earth
