File: Hotp4ck60.kicad_pcb (KiCad board)
At the start: 2 copper layers, 285 x 94.6 mm, 203 parts, among them J1 HRO_TYPE-C-31-M-12, J3 Conn_01x02_MountingPin, Q1 2N7002, SW1 RST, SW2 PWR, U1 nRF52840, U2 SRV05-4, U3 BQ24075, U4 MAX17048, Y1 32 MHz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

Commit message: Change schematic
Parts:
- removed J3: Conn_01x02_MountingPin, Connector_Molex:Molex_PicoBlade_53261-0271_1x02-1MP_P1.25mm_Horizontal
- removed R10, R12, R13: 10 kOhm, Resistor_SMD:R_0402_1005Metric
- removed R11: 100 kOhm, Resistor_SMD:R_0402_1005Metric
- removed R14: 1 MOhm, Resistor_SMD:R_0402_1005Metric
- added D65: D_Schottky, Diode_SMD:D_SOD-123, B.Cu at (91.4, 122.5)
- added J2: Conn_01x02_MountingPin, Connector_Molex:Molex_PicoBlade_53261-0271_1x02-1MP_P1.25mm_Horizontal, B.Cu at (121.3, 124.8)
- added U5: XC6206PxxxMR, Package_TO_SOT_SMD:SOT-23-3, B.Cu at (94.9, 126.9)
- C21, C23: value 4.7 uF -> 10 uF; footprint Capacitor_SMD:C_0402_1005Metric -> Capacitor_SMD:C_0805_2012Metric
- C22: value 1 uF -> 4.7 uF
- C25: value 4.7 uF -> 1 uF
- C26: value 1 uF -> 100 nF
- Q1: value 2N7002 -> AO3401A
- R3: value 47 kOhm -> 1 MOhm
- R4: value 1.5 kOhm -> 1 kOhm
- R5: value 1 kOhm -> 1.5 kOhm
- R6: value 3.9 kOhm -> 1.2 kOhm
- R7: value 10 kOhm -> 1.5 kOhm
- R8: value 1 kOhm -> 10 kOhm
- R9: value 100 Ohm -> 10 kOhm
- U3: value BQ24075 -> TP4056; footprint Package_DFN_QFN:VQFN-16-1EP_3x3mm_P0.5mm_EP1.6x1.6mm -> Package_SO:SOP-8-1EP_4.57x4.57mm_P1.27mm_EP4.57x4.45mm
- moved R9 84.0 mm to (169.4, 161.9), turned to -90 degrees
- moved R8 71.9 mm to (168.4, 161.9), turned to -90 degrees
- moved R4 71.8 mm to (161.4, 166.7), turned to 180 degrees
- moved R5 67.4 mm to (109.4, 123.9), turned to 90 degrees
- moved R3 31.1 mm to (92.8, 95.7), turned to 180 degrees
- moved C23 13.3 mm to (110.5, 120.8), turned to 0 degrees
- moved D29 11.8 mm to (91.8, 139.0)
- moved C24 11.7 mm to (91.8, 125.7), turned to 0 degrees
- moved R7 11.6 mm to (89.0, 120.8), turned to 180 degrees
- moved Q1 9.61 mm to (88.2, 123.2), turned to 90 degrees
- moved C22 7.57 mm to (96.2, 121.3)
- moved C21 7.51 mm to (94.2, 121.8)
- moved C26 7.22 mm to (101.6, 131.7), turned to 180 degrees
- moved C25 7.19 mm to (101.6, 130.6), turned to 180 degrees
- moved U3 4.73 mm to (102.8, 122.7), turned to 0 degrees
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Connections:
- C23 pad 1: VDDH -> +BATT
- C25 pad 1: +BATT -> VDD
- C26 pad 1: +BATT -> VDD
- LED2 pad 2: VDDH -> +5V
- Q1 pad 1: Net-(Q1-G) -> +5V
- Q1 pad 2: GND -> VDDH
- Q1 pad 3: /Battery/SYSOFF -> Net-(Q1-D)
- R3 pad 1: /Battery/TMR -> Earth
- R3 pad 2: GND -> GNDPWR
- R4 pad 1: /Battery/ILIM -> LED
- R4 pad 2: GND -> Net-(LED1-A)
- R5 pad 1: LED -> Net-(LED2-K)
- R5 pad 2: Net-(LED1-A) -> Net-(U3-CHRG)
- R6 pad 1: Net-(U3-ISET) -> Net-(U3-PROG)
- R7 pad 1: Net-(U3-TS) -> +5V
- R8 pad 1: Net-(LED2-K) -> VDD
- R8 pad 2: Net-(U3-~{CHG}) -> SCL
- R9 pad 1: +5V -> VDD
- R9 pad 2: Net-(Q1-G) -> SDA
- SW2 pad 1: Net-(R11-Pad1) -> +BATT
- SW2 pad 2: /Battery/SYSOFF -> Net-(Q1-D)
- SW2 pad 3: GND -> unconnected-(SW2-Pad3)
- U3 pad 1: Net-(U3-TS) -> GND
- U3 pad 2: +BATT -> Net-(U3-PROG)
- U3 pad 3: +BATT -> GND
- U3 pad 4: GND -> +5V
- U3 pad 5: GND -> +BATT
- U3 pad 6: VDDH -> unconnected-(U3-STDBY-Pad6)
- U3 pad 7: unconnected-(U3-~{PGOOD}-Pad7) -> Net-(U3-CHRG)
- U3 pad 8: GND -> +5V
- U3 pad 9: Net-(U3-~{CHG}) -> (no net)
Routing:
- net VDD: track 58.1 -> 142.2 mm, vias 6 -> 7
- net /Battery/SYSOFF: track 20.0 -> 0.00 mm, vias 2 -> 0
- net +5V: track 171.9 -> 191.8 mm, vias 1 -> 3
- net Net-(R11-Pad1): track 19.1 -> 0.00 mm, vias 2 -> 0
- net SCL: track 90.5 -> 76.0 mm
- net SDA: track 88.9 -> 74.9 mm
- net row2: track 289.7 -> 277.0 mm
- net VDDH: track 106.6 -> 118.9 mm, vias 4 -> 2
- net +BATT: track 27.9 -> 40.3 mm, vias 0 -> 2
- net Net-(LED2-K): track 3.13 -> 13.4 mm
- net GND: track 26.1 -> 18.6 mm, vias 339 -> 301
- net Net-(D29-A): track 14.8 -> 8.53 mm
- net /Battery/TMR: track 2.91 -> 0.00 mm
- net Net-(U3-PROG): track 0.00 -> 2.47 mm
- net Net-(Q1-G): track 2.46 -> 0.00 mm
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Other:
- board text added: "Off|On"
- board text removed: "On|Off"

Commit message: Update
Parts:
- removed C24, C25: 1 uF, Capacitor_SMD:C_0402_1005Metric
- removed C26: 100 nF, Capacitor_SMD:C_0402_1005Metric
- removed U5: XC6206PxxxMR, Package_TO_SOT_SMD:SOT-23-3
- C28: value 100nF -> 100 nF
- R3: value 1 MOhm -> 1.5 kOhm
- R4: value 1 kOhm -> 1.2 kOhm
- R5: value 1.5 kOhm -> 1 kOhm
- R6: value 1.2 kOhm -> 1.5 kOhm
- R7: value 1.5 kOhm -> 10 kOhm
- R9: value 10 kOhm -> 1 MOhm
- U3: footprint Package_SO:SOP-8-1EP_4.57x4.57mm_P1.27mm_EP4.57x4.45mm -> Package_SO:SOIC-8-1EP_3.9x4.9mm_P1.27mm_EP2.29x3mm
- moved R9 101.2 mm to (92.8, 95.7), turned to 180 degrees
- moved R7 97.5 mm to (177.2, 162.4), turned to 0 degrees
- moved R4 79.5 mm to (94.1, 124.4), turned to -90 degrees
- moved R5 66.2 mm to (161.2, 165.0)
- moved R3 30.2 mm to (103.5, 123.9)
- moved R6 22.0 mm to (86.2, 104.6)
- moved Q1 18.6 mm to (106.6, 126.5), turned to 0 degrees
- moved D65 17.1 mm to (87.9, 105.8)
- moved U4 16.9 mm to (129.6, 128.2), turned to 0 degrees
- moved C27 14.3 mm to (127.4, 127.7), turned to 90 degrees
- moved D29 11.8 mm to (80.2, 136.5)
- moved R8 8.99 mm to (177.2, 163.4), turned to 0 degrees
- moved SW2 7.00 mm to (104.1, 135.5), turned to -90 degrees
- moved C23 6.06 mm to (104.5, 121.8)
- moved LED1 5.94 mm to (98.0, 137.1)
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Connections:
- R3 pad 1: Earth -> Net-(LED2-K)
- R3 pad 2: GNDPWR -> Net-(U3-CHRG)
- R4 pad 1: LED -> Net-(U3-PROG)
- R4 pad 2: Net-(LED1-A) -> GND
- R5 pad 1: Net-(LED2-K) -> LED
- R5 pad 2: Net-(U3-CHRG) -> Net-(LED1-A)
- R6 pad 1: Net-(U3-PROG) -> +5V
- R7 pad 1: +5V -> VDD
- R7 pad 2: GND -> SCL
- R8 pad 2: SCL -> SDA
- R9 pad 1: VDD -> Earth
- R9 pad 2: SDA -> GNDPWR
- S43 pad 1: col1 -> col2
- S44 pad 1: col2 -> col3
- S45 pad 1: col3 -> col4
- S46 pad 1: col4 -> col5
- S47 pad 1: col5 -> col6
- S48 pad 1: col6 -> col7
- S49 pad 1: col7 -> col8
- S50 pad 1: col8 -> col9
- S57 pad 1: col5 -> col6
- S571 pad 1: col5 -> col6
- S63 pad 1: col7 -> col8
- U1 pad A10: LED -> row3
- U1 pad A8: unconnected-(U1-AIN7/P0.31-PadA8) -> LED
- U1 pad AC21: col10 -> col13
- U1 pad AD10: row1 -> SDA
- U1 pad AD12: row2 -> RST
- U1 pad AD16: col4 -> col5
- U1 pad AD18: row3 -> col7
- U1 pad AD20: col6 -> col9
- U1 pad AD22: unconnected-(U1-TRACEDATA0/P1.00-PadAD22) -> col13
- U1 pad AD8: row0 -> SCL
- U1 pad J1: row4 -> col4
- U1 pad J24: unconnected-(U1-NFC2/P0.10-PadJ24) -> col6
- U1 pad L1: unconnected-(U1-P0.06-PadL1) -> row2
- U1 pad L24: unconnected-(U1-NFC1/P0.09-PadL24) -> col8
- U1 pad N1: SDA -> row1
- U1 pad P23: col5 -> unconnected-(U1-P1.07-PadP23)
- U1 pad R1: SCL -> row0
- U1 pad R24: col9 -> col10
- U1 pad T23: col13 -> unconnected-(U1-P1.05-PadT23)
- U1 pad U1: unconnected-(U1-TRACEDATA1/P0.12-PadU1) -> row4
- U1 pad U24: col8 -> col11
- U1 pad V23: col12 -> unconnected-(U1-P1.03-PadV23)
- U1 pad W24: col7 -> col12
- U1 pad Y23: col11 -> unconnected-(U1-P1.01-PadY23)
- U3 pad 9: (no net) -> GND
Routing:
- net VDDH: track 118.9 -> 218.3 mm, vias 2 -> 6
- net VDD: track 142.2 -> 59.5 mm
- net col7: track 161.0 -> 123.7 mm
- net Earth: track 55.4 -> 21.5 mm
- net col5: track 118.7 -> 90.0 mm, vias 1 -> 2
- net col1: track 170.1 -> 152.6 mm
- net col9: track 174.8 -> 162.6 mm
- net Net-(LED1-A): track 76.3 -> 86.6 mm, vias 2 -> 4
- net row1: track 334.7 -> 325.9 mm, vias 4 -> 2
- net col8: track 169.3 -> 160.6 mm, vias 1 -> 0
- net GND: track 18.6 -> 10.6 mm, vias 301 -> 241
- net Net-(Q1-D): track 1.32 -> 9.31 mm, vias 1 -> 0
- net +5V: track 191.8 -> 199.3 mm, vias 3 -> 5
- net +BATT: track 40.3 -> 47.6 mm
- net GNDPWR: track 22.7 -> 15.6 mm
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
Commit message: Make Readme.md
Parts:
- renumbered TP1 to +3V3, TP3 to CLK, TP4 to GND, TP2 to IO
