File: Hotp4ck60_rev.A/Hotp4ck60.kicad_pcb (KiCad board)
At the start: 2 copper layers, 285 x 94.6 mm, 196 parts, among them J1 HRO_TYPE-C-31-M-12, J2 Conn_01x02_MountingPin, Q1 AO3401A, SW1 RST, SW2 PWR, U1 nRF52840, U2 SRV05-4, U3 TP4056, U4 MAX17048, Y1 32 MHz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

Commit message: Fixed path
Parts:
- removed +3V3: TestPoint, TestPoint:TestPoint_THTPad_1.0x1.0mm_Drill0.5mm
- removed C27, C28: 100 nF, Capacitor_SMD:C_0402_1005Metric
- removed CLK, GND, IO: TestPoint, TestPoint:TestPoint_THTPad_D1.0mm_Drill0.5mm
- added C24: 10 uF, Capacitor_SMD:C_0805_2012Metric, B.Cu at (104.5, 121.8)
- added C25: 100 nF, Capacitor_SMD:C_0402_1005Metric, B.Cu at (127.4, 127.7)
- added J3: Conn_01x04, Connector_PinSocket_2.54mm:PinSocket_1x04_P2.54mm_Vertical, F.Cu at (176.4, 169.9)
- added J4: Conn_01x04, Connector_PinSocket_2.54mm:PinSocket_1x04_P2.54mm_Vertical, F.Cu at (147.9, 106.4)
- C21: value 10 uF -> 100 nF; footprint Capacitor_SMD:C_0805_2012Metric -> Capacitor_SMD:C_0402_1005Metric
- C22: value 4.7 uF -> 10 uF; footprint Capacitor_SMD:C_0402_1005Metric -> Capacitor_SMD:C_0805_2012Metric
- C23: value 10 uF -> 4.7 uF; footprint Capacitor_SMD:C_0805_2012Metric -> Capacitor_SMD:C_0402_1005Metric
- moved C21 25.9 mm to (88.3, 96.8), turned to 0 degrees
- moved R6 25.4 mm to (95.7, 128.1)
- moved D65 24.5 mm to (97.3, 128.4)
- moved D18 15.9 mm to (155.6, 117.5)
- moved D44 15.9 mm to (134.9, 155.6)
- moved D48 15.9 mm to (211.1, 155.6)
- moved C23 13.0 mm to (91.6, 121.9), turned to -90 degrees
- moved D64 6.52 mm to (87.3, 100.3)
- moved Q1 6.21 mm to (100.5, 127.8), turned to 180 degrees
- moved R9 4.56 mm to (88.3, 95.8), turned to 0 degrees
- moved L5 3.95 mm to (92.0, 95.7), turned to 180 degrees
- moved F1 2.87 mm to (92.2, 96.9), turned to 0 degrees
- moved C22 2.38 mm to (93.0, 122.3)
- moved L6 1.60 mm to (89.7, 96.3)
- moved R3 0.74 mm to (103.0, 124.4), turned to 90 degrees
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Connections:
- C21 pad 1: +5V -> Earth
- C21 pad 2: GND -> GNDPWR
- C23 pad 1: +BATT -> +5V
- H8 pad 1: Earth -> GND
- R1 pad 2: GNDPWR -> GND
- R2 pad 2: GNDPWR -> GND
- U2 pad 2: +5V -> GND
- U2 pad 5: GND -> +5V
Routing:
- net VDDH: track 218.3 -> 112.0 mm, vias 6 -> 4
- net +5V: track 199.3 -> 186.9 mm, vias 5 -> 6
- net GND: track 10.6 -> 17.3 mm, vias 241 -> 197
- net Net-(Q1-D): track 9.31 -> 15.8 mm
- net col7: track 123.7 -> 130.1 mm
- net row4: track 253.1 -> 259.5 mm, vias 2 -> 3
- net GNDPWR: track 23.4 -> 17.0 mm
- net Net-(D48-A): track 7.85 -> 14.0 mm
- net Net-(D44-A): track 7.85 -> 14.0 mm
- net VBUS: track 8.37 -> 13.5 mm
- net col3: track 107.7 -> 111.7 mm
- net Net-(D18-A): track 13.3 -> 9.43 mm
- net VDD: track 59.5 -> 56.6 mm, vias 7 -> 8
- net Net-(LED2-K): track 13.3 -> 11.0 mm
- net USB-D-: track 151.4 -> 153.4 mm, vias 0 -> 1
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Other:
- outline, holes or cut-outs redrawn
- board text added: "3V3"
- board text added: "5V"
- board text added: "CLK"
- board text added: "D+"
- board text added: "D-"
- board text added: "IO"
- board text added: "⏚"

Commit message: Modified PCB designed
Parts:
- removed C21: 100 nF, Capacitor_SMD:C_0402_1005Metric
- removed D64: D_TVS, Diode_SMD:D_SOD-123F
- removed L6: BLM15PX121SN1D, Inductor_SMD:L_0402_1005Metric
- removed R9: 1 MOhm, Resistor_SMD:R_0402_1005Metric
- moved J4 61.1 mm to (86.8, 103.9), turned to 90 degrees
- moved R2 15.7 mm to (95.9, 90.9)
- moved R1 4.97 mm to (84.2, 88.8), turned to 90 degrees
- moved F1 4.16 mm to (88.1, 97.6), turned to -90 degrees
- moved L5 3.70 mm to (88.3, 95.5), turned to 0 degrees
- moved U2 1.61 mm to (91.0, 97.8)
Connections:
- J1 pad A1: GNDPWR -> GND
- J1 pad A12: GNDPWR -> GND
- J1 pad B1: GNDPWR -> GND
- J1 pad B12: GNDPWR -> GND
- J1 pad S1: Earth -> GND
- U2 pad 5: +5V -> VBUS
Routing:
- net Earth: track 23.4 -> 0.00 mm, vias 3 -> 0
- net GNDPWR: track 17.0 -> 0.00 mm, vias 2 -> 0
- net Net-(J1-CC2): track 15.9 -> 6.83 mm
- net +5V: track 186.9 -> 193.9 mm, vias 6 -> 3
- net Net-(J1-CC1): track 11.5 -> 7.71 mm
- net GND: track 17.3 -> 20.9 mm, vias 197 -> 203
- net USB-D-: track 153.4 -> 151.8 mm, vias 1 -> 0
- net USB-D+: track 153.1 -> 151.8 mm, vias 1 -> 0
- net VBUS: track 13.5 -> 12.6 mm
- net Net-(D1-A): track 32.5 -> 31.8 mm, vias 2 -> 1
- net row0: vias 0 -> 2
- removed copper zone on B.Cu, net Earth
- removed copper zone on F.Cu, net Earth
Other:
- board text added: "1.00u"
- board text added: "S2"

Commit message: Modified positions
Parts:
- removed C25: 100 nF, Capacitor_SMD:C_0402_1005Metric
- removed L5: BLM15PX121SN1D, Inductor_SMD:L_0402_1005Metric
- added C21: 10 uF, Capacitor_SMD:C_0805_2012Metric, B.Cu at (93.0, 122.3)
- C22: value 10 uF -> 4.7 uF; footprint Capacitor_SMD:C_0805_2012Metric -> Capacitor_SMD:C_0402_1005Metric
- C23: value 4.7 uF -> 10 uF; footprint Capacitor_SMD:C_0402_1005Metric -> Capacitor_SMD:C_0805_2012Metric
- C24: value 10 uF -> 100 nF; footprint Capacitor_SMD:C_0805_2012Metric -> Capacitor_SMD:C_0402_1005Metric
- moved C24 23.6 mm to (127.4, 127.7), turned to 90 degrees
- moved C23 13.0 mm to (104.5, 121.8), turned to 0 degrees
- moved F1 4.97 mm to (92.9, 96.4)
- moved C22 1.53 mm to (91.6, 121.9)
- moved U2 1.18 mm to (90.0, 98.4), turned to 90 degrees
- moved J4 0.62 mm to (86.2, 103.9)
Connections:
- C23 pad 1: +5V -> +BATT
- F1 pad 1: Net-(F1-Pad1) -> VBUS
- U2 pad 1: USB-D- -> unconnected-(U2-IO1-Pad1)
- U2 pad 4: unconnected-(U2-IO3-Pad4) -> USB-D-
- U2 pad 5: VBUS -> +5V
Routing:
- net +5V: track 193.9 -> 198.3 mm, vias 3 -> 6
- net VBUS: track 12.6 -> 8.27 mm
- net +BATT: track 48.5 -> 46.8 mm
- net Net-(F1-Pad1): track 1.50 -> 0.00 mm
- net GND: track 20.9 -> 20.0 mm, vias 203 -> 202
- net USB-D-: track 151.8 -> 152.6 mm
- net USB-D+: track 151.8 -> 151.1 mm
- net VDD: track 56.6 -> 57.2 mm

Commit message: Revision Hotp4ck 60
Parts:
- moved R2 2.08 mm to (95.9, 88.8), turned to 90 degrees
Routing:
- net GND: vias 202 -> 203
Changed lines of the file:
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@@
   )
   (footprint "Resistor_SMD:R_0402_1005Metric" (layer "B.Cu")
-    (at 95.92 90.88 -90)
+    (at 95.86 88.8 90)
     (descr "Resistor SMD 0402 (1005 Metric), square (rectangular) end terminal, IPC_7351 nominal, (Body size source: IPC-SM-782 page 72, https://www.pcb-3d.com/wordpress/wp-content/uploads/ipc-sm-782a_amendment_1_and_2.pdf), generated with kicad-footprint-generator")
     (tags "resistor")
@@
     (fp_line (start 0.525 0.27) (end 0.525 -0.27)
       (stroke (width 0.1) (type solid)) (layer "B.Fab"))
-    (pad "1" smd roundrect (at -0.51 0 270) (size 0.54 0.64) (layers "B.Cu" "B.Paste" "B.Mask") (roundrect_rratio 0.25)
+    (pad "1" smd roundrect (at -0.51 0 90) (size 0.54 0.64) (layers "B.Cu" "B.Paste" "B.Mask") (roundrect_rratio 0.25)
       (net 96 "Net-(J1-CC2)") (pintype "passive"))
-    (pad "2" smd roundrect (at 0.51 0 270) (size 0.54 0.64) (layers "B.Cu" "B.Paste" "B.Mask") (roundrect_rratio 0.25)
+    (pad "2" smd roundrect (at 0.51 0 90) (size 0.54 0.64) (layers "B.Cu" "B.Paste" "B.Mask") (roundrect_rratio 0.25)
       (net 2 "GND") (pintype "passive"))
     (model "${KICAD6_3DMODEL_DIR}/Resistor_SMD.3dshapes/R_0402_1005Metric.wrl"
@@
   (via (at 167.830002 165.039997) (size 0.6) (drill 0.3) (layers "F.Cu" "B.Cu") (net 2))
   (via (at 147.19 103.9195) (size 0.6) (drill 0.3) (layers "F.Cu" "B.Cu") (net 2))
+  (via (at 90.01 100.98) (size 0.6) (drill 0.3) (layers "F.Cu" "B.Cu") (net 2))
   (via (at 184.44 174.91) (size 0.6) (drill 0.3) (layers "F.Cu" "B.Cu") (free) (net 2))
   (via (at 153.14 175.18) (size 0.6) (drill 0.3) (layers "F.Cu" "B.Cu") (net 2))
@@
   (segment (start 175.7575 157.846296) (end 172.14 154.228796) (width 0.2) (layer "B.Cu") (net 94))
   (segment (start 159.23 126.23365) (end 159.23 110.87) (width 0.2) (layer "B.Cu") (net 94))
+  (segment (start 92.55 90.39) (end 94.78 90.39) (width 0.2) (layer "B.Cu") (net 96))
+  (segment (start 91.76 91.18) (end 92.55 90.39) (width 0.2) (layer "B.Cu") (net 96))
+  (segment (start 94.78 90.39) (end 95.86 89.31) (width 0.2) (layer "B.Cu") (net 96))
   (segment (start 91.76 93.515) (end 91.76 91.18) (width 0.2) (layer "B.Cu") (net 96))
-  (segment (start 91.76 91.18) (end 92.57 90.37) (width 0.2) (layer "B.Cu") (net 96))
-  (segment (start 92.57 90.37) (end 95.92 90.37) (width 0.2) (layer "B.Cu") (net 96))
   (segment (start 171.15 170.09) (end 171.15 170.135409) (width 0.2) (layer "B.Cu") (net 98))
   (segment (start 172.224591 171.21) (end 177.69 171.21) (width 0.2) (layer "B.Cu") (net 98))
@@
   (segment (start 165.15 169.59) (end 164.65 170.09) (width 0.15) (layer "B.Cu") (net 141))
   (segment (start 93.01 112.44) (end 89.2 108.63) (width 0.4) (layer "F.Cu") (net 144))
-  (segment (start 90.02 96.19) (end 91.11 96.19) (width 0.4) (layer "F.Cu") (net 144))
-  (segment (start 91.89 101.38) (end 87.785761 101.38) (width 0.4) (layer "F.Cu") (net 144))
-  (segment (start 92.92 98) (end 92.92 100.35) (width 0.4) (layer "F.Cu") (net 144))
+  (segment (start 92.92 100.35) (end 91.64 101.63) (width 0.4) (layer "F.Cu") (net 144))
   (segment (start 95.73 126.78) (end 94.49 125.54) (width 0.4) (layer "F.Cu") (net 144))
   (segment (start 93.01 120.37) (end 93.01 112.44) (width 0.4) (layer "F.Cu") (net 144))
+  (segment (start 91.64 101.63) (end 86.83 101.63) (width 0.4) (layer "F.Cu") (net 144))
   (segment (start 94.49 125.54) (end 94.49 121.385) (width 0.4) (layer "F.Cu") (net 144))
-  (segment (start 92.92 100.35) (end 91.89 101.38) (width 0.4) (layer "F.Cu") (net 144))
-  (segment (start 87.785761 101.38) (end 86.19 102.975761) (width 0.4) (layer "F.Cu") (net 144))
-  (segment (start 86.19 102.975761) (end 86.19 103.905) (width 0.4) (layer "F.Cu") (net 144))
+  (segment (start 90.02 96.19) (end 91.11 96.19) (width 0.4) (layer "F.Cu") (net 144))
   (segment (start 91.11 96.19) (end 92.92 98) (width 0.4) (layer "F.Cu") (net 144))
+  (segment (start 86.83 101.63) (end 86.19 102.27) (width 0.4) (layer "F.Cu") (net 144))
+  (segment (start 92.92 98) (end 92.92 100.35) (width 0.4) (layer "F.Cu") (net 144))
+  (segment (start 86.19 102.27) (end 86.19 103.905) (width 0.4) (layer "F.Cu") (net 144))
   (via (at 90.02 96.19) (size 0.6) (drill 0.3) (layers "F.Cu" "B.Cu") (net 144))
   (via (at 92.92 98) (size 0.6) (drill 0.3) (layers "F.Cu" "B.Cu") (net 144))
