File: Hotp4ck60_rev.A/Hotp4ck60.kicad_pcb (KiCad board)
At the start: 2 copper layers, 285 x 94.6 mm, 189 parts, among them J1 HRO_TYPE-C-31-M-12, J2 Conn_01x02_MountingPin, J3 Conn_01x04, J4 Conn_01x04, Q1 AO3401A, SW1 RST, SW2 PWR, U1 nRF52840, U2 SRV05-4, U3 TP4056, U4 MAX17048, Y1 32 MHz, Y2 32.768 Khz

Commit message: Create the Rev.B's gerbers and bom
Routing:
- net USB-D-: track 152.6 -> 153.7 mm
- net GND: vias 203 -> 202
Changed lines of the file:
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@@
   (via (at 166.629998 165.039999) (size 0.6) (drill 0.3) (layers "F.Cu" "B.Cu") (net 2))
   (via (at 173 176.5) (size 0.6) (drill 0.3) (layers "F.Cu" "B.Cu") (free) (net 2))
-  (via (at 87.45 102.635) (size 0.6) (drill 0.3) (layers "F.Cu" "B.Cu") (free) (net 2))
   (via (at 154.54 176.49) (size 0.6) (drill 0.3) (layers "F.Cu" "B.Cu") (free) (net 2))
   (via (at 161.047024 139.282476) (size 0.6) (drill 0.3) (layers "F.Cu" "B.Cu") (net 2))
@@
   (segment (start 87.95 90.37) (end 85.22 90.37) (width 0.2) (layer "B.Cu") (net 92))
   (segment (start 88.76 93.515) (end 88.76 91.18) (width 0.2) (layer "B.Cu") (net 92))
-  (segment (start 91.88 98.155) (end 91.88 100.46) (width 0.3) (layer "B.Cu") (net 93))
   (segment (start 90.76 95.77) (end 90.96 95.97) (width 0.3) (layer "B.Cu") (net 93))
   (segment (start 89.965 94.69) (end 90.76 94.69) (width 0.3) (layer "B.Cu") (net 93))
-  (segment (start 156.684974 107.83) (end 93.15 107.83) (width 0.2) (layer "B.Cu") (net 93))
-  (segment (start 91.27 105.95) (end 91.27 103.905) (width 0.2) (layer "B.Cu") (net 93))
-  (segment (start 159.58 110.725026) (end 159.58 126.08) (width 0.2) (layer "B.Cu") (net 93))
+  (segment (start 163.24 138.28) (end 163.24 129.74) (width 0.2) (layer "B.Cu") (net 93))
+  (segment (start 92.05 103.125) (end 91.27 103.905) (width 0.3) (layer "B.Cu") (net 93))
   (segment (start 172.5095 147.5495) (end 163.24 138.28) (width 0.2) (layer "B.Cu") (net 93))
   (segment (start 90.96 95.97) (end 90.96 97.235) (width 0.3) (layer "B.Cu") (net 93))
+  (segment (start 93.43 107.83) (end 91.27 105.67) (width 0.2) (layer "B.Cu") (net 93))
+  (segment (start 176.107863 164.432428) (end 176.107863 157.682625) (width 0.2) (layer "B.Cu") (net 93))
+  (segment (start 159.58 110.725026) (end 156.684974 107.83) (width 0.2) (layer "B.Cu") (net 93))
+  (segment (start 156.684974 107.83) (end 93.43 107.83) (width 0.2) (layer "B.Cu") (net 93))
+  (segment (start 91.27 105.67) (end 91.27 103.905) (width 0.2) (layer "B.Cu") (net 93))
+  (segment (start 171.65 165.09) (end 171.831802 165.09) (width 0.2) (layer "B.Cu") (net 93))
+  (segment (start 176.107863 157.682625) (end 172.5095 154.084262) (width 0.2) (layer "B.Cu") (net 93))
+  (segment (start 163.24 129.74) (end 159.58 126.08) (width 0.2) (layer "B.Cu") (net 93))
+  (segment (start 171.831802 165.09) (end 172.261802 165.52) (width 0.2) (layer "B.Cu") (net 93))
+  (segment (start 89.76 93.51) (end 89.76 94.485) (width 0.3) (layer "B.Cu") (net 93))
+  (segment (start 90.76 93.51) (end 90.76 95.77) (width 0.3) (layer "B.Cu") (net 93))
+  (segment (start 175.020291 165.52) (end 176.107863 164.432428) (width 0.2) (layer "B.Cu") (net 93))
+  (segment (start 89.76 94.485) (end 89.965 94.69) (width 0.3) (layer "B.Cu") (net 93))
+  (segment (start 92.05 98.325) (end 92.05 103.125) (width 0.3) (layer "B.Cu") (net 93))
+  (segment (start 172.5095 154.084262) (end 172.5095 147.5495) (width 0.2) (layer "B.Cu") (net 93))
+  (segment (start 90.96 97.235) (end 92.05 98.325) (width 0.3) (layer "B.Cu") (net 93))
   (segment (start 172.261802 165.52) (end 175.020291 165.52) (width 0.2) (layer "B.Cu") (net 93))
-  (segment (start 91.88 100.46) (end 91.27 101.07) (width 0.3) (layer "B.Cu") (net 93))
-  (segment (start 90.96 97.235) (end 91.88 98.155) (width 0.3) (layer "B.Cu") (net 93))
-  (segment (start 171.831802 165.09) (end 172.261802 165.52) (width 0.2) (layer "B.Cu") (net 93))
-  (segment (start 93.15 107.83) (end 91.27 105.95) (width 0.2) (layer "B.Cu") (net 93))
-  (segment (start 175.020291 165.52) (end 176.107863 164.432428) (width 0.2) (layer "B.Cu") (net 93))
-  (segment (start 89.76 93.51) (end 89.76 94.485) (width 0.3) (layer "B.Cu") (net 93))
-  (segment (start 172.5095 154.084262) (end 172.5095 147.5495) (width 0.2) (layer "B.Cu") (net 93))
-  (segment (start 90.76 93.51) (end 90.76 95.77) (width 0.3) (layer "B.Cu") (net 93))
-  (segment (start 171.65 165.09) (end 171.831802 165.09) (width 0.2) (layer "B.Cu") (net 93))
-  (segment (start 159.58 110.725026) (end 156.684974 107.83) (width 0.2) (layer "B.Cu") (net 93))
-  (segment (start 163.24 129.74) (end 159.58 126.08) (width 0.2) (layer "B.Cu") (net 93))
-  (segment (start 89.76 94.485) (end 89.965 94.69) (width 0.3) (layer "B.Cu") (net 93))
-  (segment (start 91.27 101.07) (end 91.27 103.905) (width 0.3) (layer "B.Cu") (net 93))
-  (segment (start 176.107863 164.432428) (end 176.107863 157.682625) (width 0.2) (layer "B.Cu") (net 93))
-  (segment (start 176.107863 157.682625) (end 172.5095 154.084262) (width 0.2) (layer "B.Cu") (net 93))
-  (segment (start 163.24 138.28) (end 163.24 129.74) (width 0.2) (layer "B.Cu") (net 93))
-  (segment (start 88.14 98.155) (end 88.14 100.46) (width 0.3) (layer "B.Cu") (net 94))
-  (segment (start 172.14 147.68365) (end 162.8895 138.43315) (width 0.2) (layer "B.Cu") (net 94))
+  (segment (start 159.58 126.08) (end 159.58 110.725026) (width 0.2) (layer "B.Cu") (net 93))
+  (segment (start 172.14 154.228796) (end 172.14 147.68365) (width 0.2) (layer "B.Cu") (net 94))
+  (segment (start 159.23 126.23365) (end 159.23 110.87) (width 0.2) (layer "B.Cu") (net 94))
+  (segment (start 162.8895 129.89315) (end 159.23 126.23365) (width 0.2) (layer "B.Cu") (net 94))
   (segment (start 90.26 92.55) (end 90.26 93.51) (width 0.3) (layer "B.Cu") (net 94))
+  (segment (start 87.97 98.325) (end 87.97 103.145) (width 0.3) (layer "B.Cu") (net 94))
   (segment (start 90.03 92.32) (end 90.26 92.55) (width 0.3) (layer "B.Cu") (net 94))
-  (segment (start 159.23 110.87) (end 156.54 108.18) (width 0.2) (layer "B.Cu") (net 94))
+  (segment (start 156.54 108.18) (end 91.26 108.18) (width 0.2) (layer "B.Cu") (net 94))
+  (segment (start 89.06 97.235) (end 87.97 98.325) (width 0.3) (layer "B.Cu") (net 94))
   (segment (start 89.475 92.32) (end 90.03 92.32) (width 0.3) (layer "B.Cu") (net 94))
   (segment (start 89.06 95.97) (end 89.06 97.235) (width 0.3) (layer "B.Cu") (net 94))
-  (segment (start 88.73 101.05) (end 88.73 103.905) (width 0.3) (layer "B.Cu") (net 94))
   (segment (start 89.26 95.77) (end 89.06 95.97) (width 0.3) (layer "B.Cu") (net 94))
-  (segment (start 162.8895 138.43315) (end 162.8895 129.89315) (width 0.2) (layer "B.Cu") (net 94))
-  (segment (start 93.005 108.18) (end 88.73 103.905) (width 0.2) (layer "B.Cu") (net 94))
+  (segment (start 174.875318 165.17) (end 175.7575 164.287818) (width 0.2) (layer "B.Cu") (net 94))
+  (segment (start 172.14 147.68365) (end 162.8895 138.43315) (width 0.2) (layer "B.Cu") (net 94))
+  (segment (start 171.65 164.59) (end 171.826776 164.59) (width 0.2) (layer "B.Cu") (net 94))
+  (segment (start 89.26 93.51) (end 89.26 95.77) (width 0.3) (layer "B.Cu") (net 94))
+  (segment (start 89.26 93.51) (end 89.26 92.535) (width 0.3) (layer "B.Cu") (net 94))
   (segment (start 175.7575 164.287818) (end 175.7575 157.846296) (width 0.2) (layer "B.Cu") (net 94))
-  (segment (start 174.875318 165.17) (end 175.7575 164.287818) (width 0.2) (layer "B.Cu") (net 94))
-  (segment (start 89.26 93.51) (end 89.26 95.77) (width 0.3) (layer "B.Cu") (net 94))
-  (segment (start 172.14 154.228796) (end 172.14 147.68365) (width 0.2) (layer "B.Cu") (net 94))
-  (segment (start 172.406776 165.17) (end 174.875318 165.17) (width 0.2) (layer "B.Cu") (net 94))
-  (segment (start 156.54 108.18) (end 93.005 108.18) (width 0.2) (layer "B.Cu") (net 94))
-  (segment (start 89.06 97.235) (end 88.14 98.155) (width 0.3) (layer "B.Cu") (net 94))
-  (segment (start 89.26 93.51) (end 89.26 92.535) (width 0.3) (layer "B.Cu") (net 94))
-  (segment (start 162.8895 129.89315) (end 159.23 126.23365) (width 0.2) (layer "B.Cu") (net 94))
   (segment (start 171.826776 164.59) (end 172.406776 165.17) (width 0.2) (layer "B.Cu") (net 94))
   (segment (start 89.26 92.535) (end 89.475 92.32) (width 0.3) (layer "B.Cu") (net 94))
-  (segment (start 171.65 164.59) (end 171.826776 164.59) (width 0.2) (layer "B.Cu") (net 94))
-  (segment (start 88.14 100.46) (end 88.73 101.05) (width 0.3) (layer "B.Cu") (net 94))
+  (segment (start 159.23 110.87) (end 156.54 108.18) (width 0.2) (layer "B.Cu") (net 94))
+  (segment (start 88.73 105.65) (end 88.73 103.905) (width 0.2) (layer "B.Cu") (net 94))
   (segment (start 175.7575 157.846296) (end 172.14 154.228796) (width 0.2) (layer "B.Cu") (net 94))
-  (segment (start 159.23 126.23365) (end 159.23 110.87) (width 0.2) (layer "B.Cu") (net 94))
+  (segment (start 172.406776 165.17) (end 174.875318 165.17) (width 0.2) (layer "B.Cu") (net 94))
+  (segment (start 162.8895 138.43315) (end 162.8895 129.89315) (width 0.2) (layer "B.Cu") (net 94))
+  (segment (start 91.26 108.18) (end 88.73 105.65) (width 0.2) (layer "B.Cu") (net 94))
+  (segment (start 87.97 103.145) (end 88.73 103.905) (width 0.3) (layer "B.Cu") (net 94))
   (segment (start 92.55 90.39) (end 94.78 90.39) (width 0.2) (layer "B.Cu") (net 96))
   (segment (start 91.76 91.18) (end 92.55 90.39) (width 0.2) (layer "B.Cu") (net 96))
@@
   (via (at 95.73 126.78) (size 0.6) (drill 0.3) (layers "F.Cu" "B.Cu") (net 144))
   (via (at 93.01 120.37) (size 0.6) (drill 0.3) (layers "F.Cu" "B.Cu") (net 144))
-  (via (at 89.2 108.63) (size 0.6) (drill 0.3) (layers "F.Cu" "B.Cu") (net 144))
+  (via (at 89.2 108.63) (size 0.6) (drill 0.4) (layers "F.Cu" "B.Cu") (net 144))
   (segment (start 94.49 121.385) (end 96.255 121.385) (width 0.4) (layer "B.Cu") (net 144))
   (segment (start 94.84 128.13) (end 95.34 127.63) (width 0.4) (layer "B.Cu") (net 144))

Commit message: unified daughterboard, MCU 추가
Parts:
- removed J4: Conn_01x04, Connector_PinSocket_2.54mm:PinSocket_1x04_P2.54mm_Vertical
- removed R1, R2: 5.1 kOhm, Resistor_SMD:R_0402_1005Metric
- removed U2: SRV05-4, PCM_marbastlib-various:SOT-23-6-routable
- added J1: Conn_01x04, Connector_JST:JST_SH_SM04B-SRSS-TB_1x04-1MP_P1.00mm_Horizontal, B.Cu at (138.8, 106.3)
- added L5: BLM15PX121SN1D, Inductor_SMD:L_0402_1005Metric, F.Cu at (169.4, 189.0)
- F1: value 750 mA -> 500mA
- J1: value HRO_TYPE-C-31-M-12 -> Conn_01x04; footprint Connector_USB:USB_C_Receptacle_HRO_TYPE-C-31-M-12 -> Connector_JST:JST_SH_SM04B-SRSS-TB_1x04-1MP_P1.00mm_Horizontal
- LED1, LED2, SW2: moved to F.Cu
- moved C4 79.4 mm to (204.5, 239.6)
- moved C11 79.4 mm to (212.2, 239.4)
- moved C17 79.4 mm to (216.0, 237.1)
- moved C5 79.4 mm to (204.2, 235.6)
- moved Y1 79.4 mm to (204.3, 237.6)
- moved AE1 79.4 mm to (208.2, 243.8)
- moved C1 79.4 mm to (207.7, 242.7)
- moved C10 79.4 mm to (205.8, 231.3)
- moved C12 79.4 mm to (207.2, 238.4)
- moved C13 79.4 mm to (207.6, 228.2)
- moved C14 79.4 mm to (206.6, 228.2)
- moved C15 79.4 mm to (213.3, 228.7)
- moved C16 79.4 mm to (216.0, 234.3)
- moved C18 79.4 mm to (206.3, 236.1)
- moved C19 79.4 mm to (215.6, 231.8)
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Connections:
- F1 pad 1: VBUS -> Net-(F1-Pad1)
- F1 pad 2: +5V -> VBUS
Routing:
- net col8: track 160.6 -> 124.4 mm
- net col10: track 193.4 -> 159.0 mm
- net +BATT: track 46.8 -> 76.0 mm, vias 2 -> 1
- net Net-(LED1-A): track 88.1 -> 115.3 mm, vias 4 -> 3
- net Net-(Q1-D): track 15.8 -> 35.4 mm, vias 0 -> 1
- net row2: track 281.0 -> 262.8 mm
- net Net-(LED2-K): track 10.7 -> 27.3 mm, vias 2 -> 1
- net +5V: track 198.7 -> 207.7 mm
- net GND: track 20.0 -> 28.9 mm, vias 202 -> 197
- net Net-(F1-Pad1): track 0.00 -> 8.27 mm, vias 0 -> 2
- net Net-(J1-CC1): track 7.71 -> 0.00 mm
- net Net-(J1-CC2): track 7.21 -> 0.00 mm
- net Net-(D29-A): track 14.1 -> 9.80 mm
- net Net-(D15-A): track 13.3 -> 14.3 mm
- net VBUS: track 8.27 -> 7.71 mm, vias 2 -> 0
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
Commit message: 리비젼A 수정
Parts:
- removed the J1 at (90.0, 89.5)
- removed the J1 at (138.8, 106.3)
- removed J2: Conn_01x02_MountingPin, Connector_Molex:Molex_PicoBlade_53261-0271_1x02-1MP_P1.25mm_Horizontal
- removed L5: BLM15PX121SN1D, Inductor_SMD:L_0402_1005Metric
- added J1: Conn_01x05_Pin, Connector_PinHeader_2.54mm:PinHeader_1x05_P2.54mm_Vertical, F.Cu at (209.6, 125.5)
- H8: footprint amtra5_outline:60_Outline-Modded-Type-C -> Hotp4ck:Neo60_2
- SW2: value PWR -> SW_DIP_x01; footprint marbastlib-various:SW_MSK12C02-HB -> Hotp4ck:SW_DIP_HOTP4CK
- moved C1 68.0 mm to (213.8, 175.0), turned to -90 degrees
- moved C17 67.4 mm to (221.8, 169.9)
- moved C7 67.4 mm to (215.6, 158.5)
- moved C11 67.4 mm to (218.1, 172.2)
- moved C15 67.4 mm to (219.2, 161.5)
- moved C19 67.4 mm to (221.5, 164.6)
- moved C3 67.4 mm to (215.3, 171.2)
- moved C4 67.4 mm to (210.4, 172.4)
- moved C5 67.4 mm to (210.0, 168.4)
- moved C6 67.4 mm to (214.5, 158.5)
- moved C8 67.4 mm to (220.5, 161.0)
- moved C9 67.4 mm to (210.4, 163.5)
- moved R5 67.4 mm to (209.4, 165.0)
- moved Y1 67.4 mm to (210.2, 170.4)
- moved C13 67.4 mm to (213.5, 161.0)
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Connections:
- F1 pad 1: Net-(F1-Pad1) -> VBUS
- F1 pad 2: VBUS -> +5V
- U1 pad A10: row3 -> col5
- U1 pad A12: col0 -> col4
- U1 pad A16: col2 -> col3
- U1 pad A20: col3 -> col6
- U1 pad AC21: col13 -> unconnected-(U1-P0.25-PadAC21)
- U1 pad AD16: col5 -> unconnected-(U1-P0.20-PadAD16)
- U1 pad AD18: col7 -> unconnected-(U1-P0.22-PadAD18)
- U1 pad AD22: col13 -> unconnected-(U1-TRACEDATA0/P1.00-PadAD22)
- U1 pad B13: unconnected-(U1-AIN1/P0.03-PadB13) -> col0
- U1 pad B15: unconnected-(U1-P1.14-PadB15) -> col2
- U1 pad G1: unconnected-(U1-P0.26-PadG1) -> row3
- U1 pad J1: col4 -> col7
- U1 pad J24: col6 -> col8
- U1 pad L24: col8 -> col10
- U1 pad R24: col10 -> col11
- U1 pad U24: col11 -> col12
- U1 pad W24: col12 -> col13
Routing:
- net row0: track 296.4 -> 19.8 mm, vias 2 -> 1
- net +5V: track 207.7 -> 8.71 mm, vias 6 -> 0
- net USB-D-: track 153.7 -> 11.2 mm
- net USB-D+: track 151.1 -> 11.8 mm
- net Net-(LED1-A): track 115.3 -> 3.92 mm, vias 3 -> 0
- net VDDH: track 112.0 -> 12.2 mm, vias 4 -> 1
- net col9: track 162.2 -> 71.3 mm
- net +BATT: track 76.0 -> 0.00 mm, vias 1 -> 0
- net SDA: track 83.0 -> 12.5 mm, vias 2 -> 0
- net SCL: track 82.5 -> 12.2 mm, vias 2 -> 0
- net row1: track 325.1 -> 267.1 mm, vias 4 -> 1
- net col2: track 130.3 -> 185.9 mm, vias 0 -> 1
- net col3: track 111.7 -> 163.5 mm, vias 0 -> 1
- net col7: track 130.1 -> 79.8 mm, vias 1 -> 0
- net col11: track 217.9 -> 167.8 mm, vias 1 -> 0
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Other:
- board size 285 x 94.6 mm -> 284.7 x 94.2 mm

Commit message: 배선 완료
Parts:
- removed the C1 at (213.8, 175.0)
- removed J3: Conn_01x04, Connector_PinSocket_2.54mm:PinSocket_1x04_P2.54mm_Vertical
- removed LED2: Yellow, LED_SMD:LED_0603_1608Metric
- removed SW1: RST, marbastlib-various:SW_SPST_SKQG_WithStem
- added C24: 4u7, Capacitor_SMD:C_0402_1005Metric, B.Cu at (110.9, 124.6)
- added C25: 1u, Capacitor_SMD:C_0402_1005Metric, B.Cu at (111.9, 124.6)
- added C26: 4u7, Capacitor_SMD:C_0402_1005Metric, B.Cu at (104.0, 124.6)
- added C27: 1u, Capacitor_SMD:C_0402_1005Metric, B.Cu at (105.0, 124.6)
- added J2: Conn_01x05_Socket, Connector_PinSocket_2.54mm:PinSocket_1x05_P2.54mm_Vertical, F.Cu at (233.0, 163.5)
- added L2: 4.7 nH, Inductor_SMD:L_0402_1005Metric, B.Cu at (215.3, 175.3)
- added R1: 68k, Resistor_SMD:R_0805_2012Metric, B.Cu at (107.4, 130.2)
- added R10: 1k, Resistor_SMD:R_0402_1005Metric, B.Cu at (86.6, 142.4)
- added R2: 1k5, Resistor_SMD:R_0402_1005Metric, B.Cu at (111.4, 126.1)
- added R9: 1k, Resistor_SMD:R_0402_1005Metric, B.Cu at (88.1, 142.4)
- added U2: BQ24075RGT, Package_DFN_QFN:VQFN-16-1EP_3x3mm_P0.5mm_EP1.6x1.6mm, B.Cu at (108.1, 125.1)
- C1: renamed from C2; value 0.5 pF -> 1.2 pF
- C2: renamed from C3; value 0.8 pF -> 1 pF
- C21, C23: value 10 uF -> 4u7; footprint Capacitor_SMD:C_0805_2012Metric -> Capacitor_SMD:C_0402_1005Metric
- C22: value 4.7 uF -> 4u7
- LED1: value Blue -> LED_MHT151RGBCT; footprint LED_SMD:LED_0603_1608Metric -> PCM_marbastlib-various:LED_1206R; moved to B.Cu
- R3: value 1.5 kOhm -> 2k2
- R4: value 1.2 kOhm -> 10k
- R8: renamed from R5; value 1 kOhm -> 1k
- U3: value TP4056 -> SRV05-4; footprint Package_SO:SOIC-8-1EP_3.9x4.9mm_P1.27mm_EP2.29x3mm -> PCM_marbastlib-various:SOT-23-6-routable
- moved U3 152.4 mm to (214.3, 114.9), turned to 180 degrees
- moved R8 121.8 mm to (89.7, 142.4), turned to -90 degrees
- moved F1 111.6 mm to (204.1, 106.4), turned to 180 degrees
- moved R5 26.7 mm to (121.7, 124.2), turned to -90 degrees
- moved U4 25.6 mm to (104.0, 128.3), turned to -90 degrees
- moved C7 23.9 mm to (103.5, 126.1), turned to 180 degrees
- moved D65 22.8 mm to (119.9, 125.3)
- moved D1 21.9 mm to (89.2, 98.4)
- moved D15 19.9 mm to (77.7, 119.6), turned to 90 degrees
- moved D21 19.6 mm to (196.8, 119.6), turned to 90 degrees
- moved C22 19.5 mm to (110.0, 128.2)
- moved J1 19.2 mm to (209.2, 106.4)
- moved C21 18.9 mm to (111.0, 128.2)
- moved Q1 15.9 mm to (116.2, 125.4)
- moved LED1 13.2 mm to (88.1, 139.7), turned to 180 degrees
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- renumbered C4 to C3, C5 to C4, C6 to C5, C7 to C6, C24 to C7, L2 to L3, L3 to L4, L4 to L5, R6 to R5, R7 to R6, R8 to R7
Connections:
- C1 pad 2: Net-(AE1-Pad1) -> Net-(C1-Pad2)
- C23 pad 1: +BATT -> +5V
- L1 pad 1: Net-(AE1-Pad1) -> Net-(C1-Pad2)
- LED1 pad 1: GND -> VDD
- LED1 pad 2: Net-(LED1-A) -> Net-(LED1-BK)
- R3 pad 2: Net-(U3-CHRG) -> GND
- R4 pad 1: Net-(U3-PROG) -> Net-(U2-TS)
- R8 pad 1: LED -> Net-(LED1-BK)
- R8 pad 2: Net-(LED1-A) -> LED_B
- U1 pad A10: col5 -> col4
- U1 pad A12: col4 -> LED_B
- U1 pad A8: LED -> col5
- U1 pad AD16: unconnected-(U1-P0.20-PadAD16) -> col9
- U1 pad AD20: col9 -> unconnected-(U1-P0.24-PadAD20)
- U3 pad 1: GND -> USB-D+
- U3 pad 2: Net-(U3-PROG) -> GND
- U3 pad 3: GND -> unconnected-(U3-IO2-Pad3)
- U3 pad 4: +5V -> unconnected-(U3-IO3-Pad4)
- U3 pad 5: +BATT -> VBUS
- U3 pad 6: unconnected-(U3-STDBY-Pad6) -> USB-D-
Routing:
- net row0: track 19.8 -> 319.3 mm, vias 1 -> 2
- net +5V: track 8.71 -> 265.5 mm, vias 0 -> 6
- net SDA: track 12.5 -> 166.3 mm, vias 0 -> 4
- net SCL: track 12.2 -> 164.9 mm, vias 0 -> 4
- net LED_B: track 0.00 -> 146.5 mm
- net VDDH: track 12.2 -> 157.3 mm, vias 1 -> 2
- net +BATT: track 0.00 -> 144.6 mm, vias 0 -> 1
- net VDD: track 73.3 -> 214.6 mm, vias 8 -> 10
- net USB-D-: track 11.2 -> 70.2 mm, vias 0 -> 2
- net USB-D+: track 11.8 -> 70.6 mm, vias 0 -> 2
- net ~{CHG}: track 0.00 -> 44.8 mm, vias 0 -> 4
- net col9: track 71.3 -> 114.2 mm, vias 1 -> 3
- net row1: track 267.1 -> 303.7 mm, vias 1 -> 4
- net Net-(Q1-D): track 3.00 -> 26.0 mm, vias 1 -> 3
- net RST: track 4.30 -> 27.1 mm, vias 0 -> 2
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- added copper zone on B.Cu, net +BATT
- added copper zone on B.Cu, net VDDH
Other:
- board text removed: ""
