File: Hotp4ck60_rev.A/Hotpacky60_Matrix.kicad_sch (KiCad schematic)
At the start: 127 parts

Commit message: 리비젼A 수정
Parts:
- renumbered S1 to S10, S1 to S11, S1 to S12, S1 to S13, S60 to S14, S2 to S15, S1 to S16, S1 to S17, S1 to S18, S1 to S19, S1 to S2, S1 to S20, S1 to S21, S1 to S22, S1 to S23, S1 to S24, S1 to S25, S1 to S26, S1 to S27, S2 to S28, S2 to S29, S1 to S3, S1 to S30, S1 to S31, S1 to S32, S1 to S33, S1 to S34, S1 to S35, S1 to S36, S1 to S37, S1 to S38, S1 to S39, S1 to S4, S1 to S40, S62 to S41, S62 to S42, S1 to S43, S1 to S44, S1 to S45, S1 to S46, S1 to S47, S1 to S48, S1 to S49, S1 to S5, S1 to S50, S1 to S51, S1 to S52, S58 to S53, S5 to S54, S5 to S55, S5 to S56, S36 to S57, S58 to S571, S5 to S58, S5 to S59, S1 to S6, S5 to S60, S5 to S61, S5 to S62, S62 to S63, S1 to S7, S1 to S8, S1 to S9
Changed lines of the file:
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@@
 (kicad_sch
-	(version 20231120)
+	(version 20250114)
 	(generator "eeschema")
-	(generator_version "8.0")
+	(generator_version "9.0")
 	(paper "A4")
 	(junction
@@
 		(on_board yes)
 		(dnp no)
-		(property "Reference" "S62"
+		(property "Reference" "S63"
 			(at 168.91 97.79 90)
 			(effects
@@
 		(on_board yes)
 		(dnp no)
-		(property "Reference" "S1"
+		(property "Reference" "S2"
 			(at 53.34 31.75 90)
 			(effects
@@
 		(on_board yes)
 		(dnp no)
-		(property "Reference" "S1"
+		(property "Reference" "S45"
 			(at 102.87 81.28 90)
 			(effects
@@
 		(on_board yes)
 		(dnp no)
-		(property "Reference" "S1"
+		(property "Reference" "S36"
 			(at 152.4 64.77 90)
 			(effects
@@
 		(on_board yes)
 		(dnp no)
-		(property "Reference" "S2"
+		(property "Reference" "S29"
 			(at 36.83 64.77 90)
 			(effects
@@
 		(on_board yes)
 		(dnp no)
-		(property "Reference" "S5"
+		(property "Reference" "S60"
 			(at 234.95 97.79 90)
 			(effects
@@
 		(on_board yes)
 		(dnp no)
-		(property "Reference" "S1"
+		(property "Reference" "S35"
 			(at 135.89 64.77 90)
 			(effects
@@
 		(on_board yes)
 		(dnp no)
-		(property "Reference" "S1"
+		(property "Reference" "S26"
 			(at 218.44 48.26 90)
 			(effects
@@
 		(on_board yes)
 		(dnp no)
-		(property "Reference" "S5"
+		(property "Reference" "S56"
 			(at 69.85 97.79 90)
 			(effects
@@
 		(on_board yes)
 		(dnp no)
-		(property "Reference" "S1"
+		(property "Reference" "S52"
 			(at 218.44 81.28 90)
 			(effects
@@
 		(on_board yes)
 		(dnp no)
-		(property "Reference" "S5"
+		(property "Reference" "S54"
 			(at 36.83 97.79 90)
 			(effects
@@
 		(on_board yes)
 		(dnp no)
-		(property "Reference" "S58"
+		(property "Reference" "S571"
 			(at 135.89 110.49 90)
 			(effects
@@
 		(on_board yes)
 		(dnp no)
-		(property "Reference" "S1"
+		(property "Reference" "S50"
 			(at 185.42 81.28 90)
 			(effects
@@
 		(on_board yes)
 		(dnp no)
-		(property "Reference" "S1"
+		(property "Reference" "S43"
 			(at 69.85 81.28 90)
 			(effects
@@
 		(on_board yes)
 		(dnp no)
-		(property "Reference" "S1"
+		(property "Reference" "S34"
 			(at 119.38 64.77 90)
 			(effects
@@
 		(on_board yes)
 		(dnp no)
-		(property "Reference" "S1"
+		(property "Reference" "S6"
 			(at 119.38 31.75 90)
 			(effects
@@
 		(on_board yes)
 		(dnp no)
-		(property "Reference" "S1"
+		(property "Reference" "S38"
 			(at 185.42 64.77 90)
 			(effects
@@
 		(on_board yes)
 		(dnp no)
-		(property "Reference" "S1"
+		(property "Reference" "S8"
 			(at 152.4 31.75 90)
 			(effects
@@
 		(on_board yes)
 		(dnp no)
-		(property "Reference" "S36"
+		(property "Reference" "S57"
 			(at 132.08 97.79 90)
 			(effects
@@
 		(on_board yes)
 		(dnp no)
-		(property "Reference" "S1"
+		(property "Reference" "S27"
 			(at 234.95 48.26 90)
 			(effects
@@
 		(on_board yes)
 		(dnp no)
-		(property "Reference" "S62"
+		(property "Reference" "S42"
 			(at 36.83 81.28 90)
 			(effects
@@
 		(on_board yes)
 		(dnp no)
-		(property "Reference" "S1"
+		(property "Reference" "S32"
 			(at 86.36 64.77 90)
 			(effects
@@
 		(on_board yes)
 		(dnp no)
-		(property "Reference" "S1"
+		(property "Reference" "S46"
 			(at 119.38 81.28 90)
 			(effects
@@
 		(on_board yes)
 		(dnp no)
-		(property "Reference" "S1"
+		(property "Reference" "S51"
 			(at 201.93 81.28 90)
 			(effects
@@
 		(on_board yes)
 		(dnp no)
-		(property "Reference" "S1"
+		(property "Reference" "S30"
 			(at 53.34 64.77 90)
 			(effects
@@
 		(on_board yes)
 		(dnp no)
-		(property "Reference" "S1"
+		(property "Reference" "S23"
 			(at 168.91 48.26 90)
 			(effects
@@
 		(on_board yes)
 		(dnp no)
-		(property "Reference" "S1"
+		(property "Reference" "S49"
 			(at 168.91 81.28 90)
 			(effects
@@
 		(on_board yes)
 		(dnp no)
-		(property "Reference" "S1"
+		(property "Reference" "S39"
 			(at 201.93 64.77 90)
 			(effects
@@
 		(on_board yes)
 		(dnp no)
-		(property "Reference" "S1"
+		(property "Reference" "S33"
 			(at 102.87 64.77 90)
 			(effects
@@
 		(on_board yes)
 		(dnp no)
-		(property "Reference" "S1"
+		(property "Reference" "S48"
 			(at 152.4 81.28 90)
 			(effects
@@
 		(on_board yes)
 		(dnp no)
-		(property "Reference" "S58"
+		(property "Reference" "S53"
 			(at 251.46 81.28 90)
 			(effects
@@
 		(on_board yes)
 		(dnp no)
-		(property "Reference" "S1"
+		(property "Reference" "S19"
 			(at 102.87 48.26 90)
 			(effects
@@
 		(on_board yes)
 		(dnp no)
-		(property "Reference" "S60"
+		(property "Reference" "S14"
 			(at 251.46 31.75 90)
 			(effects
@@
 		(on_board yes)
 		(dnp no)
-		(property "Reference" "S1"
+		(property "Reference" "S40"
 			(at 218.44 64.77 90)
 			(effects
@@
 		(on_board yes)
 		(dnp no)
-		(property "Reference" "S1"
+		(property "Reference" "S25"
 			(at 201.93 48.26 90)
 			(effects
@@
 		(on_board yes)
 		(dnp no)
-		(property "Reference" "S5"
+		(property "Reference" "S55"
 			(at 53.34 97.79 90)
 			(effects
@@
 		(on_board yes)
 		(dnp no)
-		(property "Reference" "S1"
+		(property "Reference" "S4"
 			(at 86.36 31.75 90)
 			(effects
@@
 		(on_board yes)
 		(dnp no)
-		(property "Reference" "S1"
+		(property "Reference" "S44"
 			(at 86.36 81.28 90)
 			(effects
@@
 		(on_board yes)
 		(dnp no)
-		(property "Reference" "S5"
+		(property "Reference" "S59"
 			(at 218.44 97.79 90)
 			(effects
@@
 		(on_board yes)
 		(dnp no)
-		(property "Reference" "S1"
+		(property "Reference" "S5"
 			(at 102.87 31.75 90)
 			(effects
@@
 		(on_board yes)
 		(dnp no)
-		(property "Reference" "S1"
+		(property "Reference" "S13"
 			(at 234.95 31.75 90)
 			(effects
@@
 		(on_board yes)
 		(dnp no)
-		(property "Reference" "S1"
+		(property "Reference" "S21"
 			(at 135.89 48.26 90)
 			(effects
@@
 		(on_board yes)
 		(dnp no)
-		(property "Reference" "S2"
+		(property "Reference" "S28"
 			(at 251.46 48.26 90)
 			(effects
@@
 		(on_board yes)
 		(dnp no)
-		(property "Reference" "S5"
+		(property "Reference" "S62"
 			(at 86.36 97.79 90)
 			(effects
@@
 		(on_board yes)
 		(dnp no)
-		(property "Reference" "S1"
+		(property "Reference" "S18"
 			(at 86.36 48.26 90)
 			(effects
@@
 		(on_board yes)
 		(dnp no)
-		(property "Reference" "S1"
+		(property "Reference" "S7"
 			(at 135.89 31.75 90)
 			(effects
@@
 		(on_board yes)
 		(dnp no)
-		(property "Reference" "S1"
+		(property "Reference" "S24"
 			(at 185.42 48.26 90)
 			(effects
@@
 		(on_board yes)
 		(dnp no)
-		(property "Reference" "S1"
+		(property "Reference" "S9"
 			(at 168.91 31.75 90)
 			(effects
@@
 		(on_board yes)
 		(dnp no)
-		(property "Reference" "S5"
+		(property "Reference" "S58"
 			(at 201.93 97.79 90)
 			(effects
@@
 		(on_board yes)
 		(dnp no)
-		(property "Reference" "S1"
+		(property "Reference" "S37"
 			(at 168.91 64.77 90)
 			(effects
@@
 		(on_board yes)
 		(dnp no)
-		(property "Reference" "S2"
+		(property "Reference" "S15"
 			(at 36.83 48.26 90)
 			(effects
@@
 		(on_board yes)
 		(dnp no)
-		(property "Reference" "S1"
+		(property "Reference" "S3"
 			(at 69.85 31.75 90)
 			(effects
@@
 		(on_board yes)
 		(dnp no)
-		(property "Reference" "S1"
+		(property "Reference" "S47"
 			(at 135.89 81.28 90)
 			(effects
@@
 		(on_board yes)
 		(dnp no)
-		(property "Reference" "S1"
+		(property "Reference" "S20"
 			(at 119.38 48.26 90)
 			(effects
@@
 		(on_board yes)
 		(dnp no)
-		(property "Reference" "S1"
+		(property "Reference" "S10"
 			(at 185.42 31.75 90)
 			(effects
@@
 		(on_board yes)
 		(dnp no)
-		(property "Reference" "S1"
+		(property "Reference" "S16"
 			(at 53.34 48.26 90)
 			(effects
@@
 		(on_board yes)
 		(dnp no)
-		(property "Reference" "S62"
+		(property "Reference" "S41"
 			(at 251.46 64.77 90)
 			(effects
@@
 		(on_board yes)
 		(dnp no)
-		(property "Reference" "S1"
+		(property "Reference" "S12"
 			(at 218.44 31.75 90)
 			(effects
@@
 		(on_board yes)
 		(dnp no)
-		(property "Reference" "S5"
+		(property "Reference" "S61"
 			(at 251.46 97.79 90)
 			(effects
@@
 		(on_board yes)
 		(dnp no)
-		(property "Reference" "S1"
+		(property "Reference" "S22"
 			(at 152.4 48.26 90)
 			(effects
@@
 		(on_board yes)
 		(dnp no)
-		(property "Reference" "S1"
+		(property "Reference" "S11"
 			(at 201.93 31.75 90)
 			(effects
@@
 		(on_board yes)
 		(dnp no)
-		(property "Reference" "S1"
+		(property "Reference" "S31"
 			(at 69.85 64.77 90)
 			(effects
@@
 		(on_board yes)
 		(dnp no)
-		(property "Reference" "S1"
+		(property "Reference" "S17"
 			(at 69.85 48.26 90)
 			(effects
