File: Hotp4ck60_rev.B/Hotp4ck60.kicad_pcb (KiCad board)
At the start: 2 copper layers, 285 x 94.6 mm, 188 parts, among them J1 JST, J2 Conn_01x02_MountingPin, Q1 2N7002, SW1 Reset, SW2 PWR, U1 nRF52840, U2 BQ24075, U3 MAX17048, Y1 32 MHz, Y2 32.768 Khz

Commit message: Create the Rev.B's gerbers and bom
Parts:
- moved C9 8.06 mm to (160.0, 174.5), turned to -90 degrees
- moved SW1 2.02 mm to (189.7, 173.9)
- moved L1 1.46 mm to (166.6, 182.2)
- moved C2 1.44 mm to (166.2, 183.8)
- moved C3 1.44 mm to (166.2, 180.7)
- moved R1 0.81 mm to (157.9, 173.5)
- moved L3 0.73 mm to (159.5, 173.0), turned to 180 degrees
- moved C11 0.22 mm to (168.3, 181.1)
- moved C1 0.17 mm to (165.8, 186.6)
Routing:
- net Net-(AE1-Pad1): track 0.88 -> 4.84 mm
- net Net-(SW2-A): track 70.0 -> 71.9 mm
- net RST: track 23.5 -> 25.0 mm
- net SYSOFF: track 81.2 -> 82.1 mm
- net LED: track 6.79 -> 7.72 mm
- net Net-(LED1-A): track 83.7 -> 82.8 mm
- net col4: track 85.2 -> 85.7 mm
- net GND: track 17.1 -> 16.9 mm, vias 121 -> 122

Commit message: Change to daugtherboard
Parts:
- removed AE1: 2.4 GHz ANT, RF_Antenna:Texas_SWRA117D_2.4GHz_Right
- removed C15, C19, C20, C21, C22, C23: 4.7 uF, Capacitor_SMD:C_0402_1005Metric
- removed C16, C17, C18, C24: 100 nF, Capacitor_SMD:C_0402_1005Metric
- removed L1: 4.7 nH, Inductor_SMD:L_0402_1005Metric
- removed L3: 15 nH, Inductor_SMD:L_0402_1005Metric
- removed L4: 10 uH, Inductor_SMD:L_0603_1608Metric
- removed LED2: orange, LED_SMD:LED_0603_1608Metric
- removed R1: 1 kOhm, Resistor_SMD:R_0402_1005Metric
- removed R2: 47 kOhm, Resistor_SMD:R_0402_1005Metric
- removed SW1: Reset, marbastlib-various:SW_SPST_SKQG_WithStem
- removed SW2: PWR, PCM_marbastlib-various:SW_MSK12C02-HB
- removed Y2: 32.768 Khz, Crystal:Crystal_SMD_2012-2Pin_2.0x1.2mm
- added PWR1: PWR, PCM_marbastlib-various:SW_MSK12C02-HB, B.Cu at (219.8, 203.2)
- added R12: 100 Ohm, Resistor_SMD:R_0402_1005Metric, B.Cu at (236.5, 213.4)
- added R13: 10 kOhm, Resistor_SMD:R_0402_1005Metric, B.Cu at (236.5, 215.4)
- added R14: 100 kOhm, Resistor_SMD:R_0402_1005Metric, B.Cu at (236.5, 217.3)
- added RST1: RST, PCM_marbastlib-various:SW_T1A2QR, B.Cu at (171.0, 233.4)
- added U5: 74LVC1G11, Package_TO_SOT_SMD:SOT-363_SC-70-6, B.Cu at (153.2, 210.7)
- C1: value NC -> 4u7
- C10: value 47 nF -> 4u7; footprint Capacitor_SMD:C_0603_1608Metric -> Capacitor_SMD:C_0402_1005Metric
- C11: value 820 pF -> 4u7
- C12: value 100 pF -> 12p
- C13: value 100 nF -> 12p
- C14: value 1 uF -> 100n
- C2: value 0.5 pF -> 4u7
- C3: value 0.8 pF -> 1u
- C4, C7: value 12 pF -> 4u7
- C5: value 12 pF -> 1u
- C6: value 12 pF -> 100n
- C8: value 4.7 uF -> 1u
- C9: value 1 uF -> 1u
- J3: moved to B.Cu
- LED1: value Blue -> IND; footprint LED_SMD:LED_0603_1608Metric -> PCM_marbastlib-various:LED_1206R
- R10, R11: value 10 kOhm -> 1k
- R3: value 1.1 kOhm -> 10k
- R4: value 1 kOhm -> 47k
- R5: value 10 kOhm -> 1k5
- R6: value 1.5 kOhm -> 2k2
- R7: value 100 Ohm -> 10k
- R8: value 10 kOhm -> 10k
- R9: value 100 kOhm -> 1k
- U1: value nRF52840 -> MAX17048; footprint Package_DFN_QFN:Nordic_AQFN-73-1EP_7x7mm_P0.5mm -> Package_DFN_QFN:DFN-8-1EP_2x2mm_P0.5mm_EP0.6x1.2mm
- U3: value MAX17048 -> nRF52840_E73-2G4M08S1C; footprint Package_DFN_QFN:DFN-8-1EP_2x2mm_P0.5mm_EP0.7x1.3mm -> PCM_marbastlib-various:nRF52840_E73-2G4M08S1C
- Y1: value 32 MHz -> 32.768 KHz; footprint Crystal:Crystal_SMD_2016-4Pin_2.0x1.6mm -> Crystal:Crystal_SMD_2012-2Pin_2.0x1.2mm
- moved U2 115.7 mm to (251.9, 220.8), turned to 180 degrees
- moved Q1 113.7 mm to (245.7, 224.9), turned to -90 degrees
- moved R9 113.7 mm to (90.9, 218.3), turned to 180 degrees
- moved R3 106.9 mm to (236.5, 220.2), turned to 180 degrees
- moved R6 105.3 mm to (239.4, 213.4), turned to 180 degrees
- moved R5 104.7 mm to (236.5, 224.2), turned to 180 degrees
- moved R4 103.9 mm to (236.5, 222.2), turned to 180 degrees
- moved J2 99.3 mm to (238.4, 203.5)
- moved R11 95.3 mm to (90.9, 222.3)
- moved R10 93.7 mm to (90.9, 220.3)
- moved C5 78.9 mm to (228.9, 218.2)
- moved LED1 77.9 mm to (83.0, 219.2), turned to 180 degrees
- moved C6 77.2 mm to (223.1, 219.6)
- moved C4 75.4 mm to (228.9, 216.2)
- moved C7 74.0 mm to (226.1, 212.2), turned to 180 degrees
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- renumbered D62 to D57, D57 to D58, D58 to D59, D59 to D60, D60 to D61, D61 to D62, S62 to S57, S57 to S58, S63 to S59, S58 to S60, S59 to S61, S60 to S62, S61 to S63, S571 to S64
Connections:
- C1 pad 1: GND -> +5V
- C1 pad 2: Net-(AE1-Pad1) -> GND
- C10 pad 1: DEC4_6 -> +5V
- C11 pad 1: DEC5 -> +VSW
- C12 pad 1: DEC3 -> Net-(U3-P0.00/XL1)
- C13 pad 1: DEC1 -> Net-(U3-P0.01/XL2)
- C2 pad 1: GND -> +5V
- C2 pad 2: Net-(AE1-Pad1) -> GND
- C3 pad 1: GND -> +5V
- C3 pad 2: Net-(U1-ANT) -> GND
- C4 pad 1: GND -> +VSW
- C4 pad 2: Net-(U1-XC1) -> GND
- C5 pad 1: Net-(U1-XC2) -> +VSW
- C6 pad 1: Net-(U1-XL1/P0.00) -> +BATT
- C7 pad 1: Net-(U1-XL2/P0.01) -> +BATT
- C8 pad 1: VDDH -> +BATT
- C9 pad 1: DEC4_6 -> VDD
- L2 pad 1: DCC -> DCCH
- L2 pad 2: Net-(L2-Pad2) -> VDD
- LED1 pad 1: GND -> VDD
- LED1 pad 2: Net-(LED1-A) -> Net-(LED1-BK)
- R10 pad 1: VDD -> Net-(LED1-GK)
- R10 pad 2: SCL -> LED_G
- R11 pad 1: VDD -> Net-(LED1-RK)
- R11 pad 2: SDA -> ~{CHG}
- R3 pad 1: /Battery/ILIM -> Net-(U2-TS)
- R4 pad 1: Net-(U2-ISET) -> /TMR
- R5 pad 1: Net-(U2-TS) -> /ILIM
- R6 pad 1: Net-(LED2-K) -> Net-(U2-ISET)
- R6 pad 2: Net-(U2-~{CHG}) -> GND
- R7 pad 1: +5V -> VDD
- R7 pad 2: Net-(Q1-G) -> SDA
- R8 pad 1: Net-(Q1-G) -> VDD
- R8 pad 2: GND -> SCL
- R9 pad 1: Net-(SW2-A) -> Net-(LED1-BK)
- R9 pad 2: +BATT -> LED_B
- U2 pad 10: VDDH -> +VSW
- U2 pad 11: VDDH -> +VSW
- U2 pad 12: /Battery/ILIM -> /ILIM
- U2 pad 14: /Battery/TMR -> /TMR
- U2 pad 5: VDDH -> GND
- U2 pad 6: GND -> +VSW
- U2 pad 9: Net-(U2-~{CHG}) -> ~{CHG}
- U3 pad 1: GND -> unconnected-(U3-P1.11-Pad1)
- U3 pad 2: +BATT -> unconnected-(U3-P1.10-Pad2)
- U3 pad 3: +BATT -> c06
- U3 pad 4: GND -> c07
- U3 pad 5: ALERT -> GND
- U3 pad 6: GND -> unconnected-(U3-P1.13-Pad6)
- U3 pad 7: SCL -> c08
- U3 pad 8: SDA -> c09
- U3 pad 9: GND -> c10
- Y1 pad 1: Net-(U1-XC1) -> Net-(U3-P0.01/XL2)
- Y1 pad 2: GND -> Net-(U3-P0.00/XL1)
Routing:
- net row0: track 310.2 -> 0.00 mm, vias 2 -> 0
- net row1: track 290.8 -> 0.00 mm, vias 4 -> 0
- net row4: track 280.9 -> 0.00 mm, vias 4 -> 0
- net col13: track 271.5 -> 0.00 mm
- net row2: track 269.8 -> 0.00 mm, vias 4 -> 0
- net col12: track 241.2 -> 0.00 mm
- net col11: track 217.0 -> 0.00 mm
- net col10: track 196.9 -> 0.00 mm
- net row3: track 179.5 -> 0.00 mm, vias 2 -> 0
- net col0: track 175.9 -> 0.00 mm
- net col8: track 161.8 -> 0.00 mm
- net col9: track 161.5 -> 0.00 mm
- net col1: track 151.0 -> 0.00 mm
- net VDDH: track 137.6 -> 0.00 mm, vias 7 -> 0
- net col2: track 130.2 -> 0.00 mm
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Other:
- outline, holes or cut-outs redrawn

Commit message: place parts and trace connect
Parts:
- removed PWR1: PWR, PCM_marbastlib-various:SW_MSK12C02-HB
- removed Q1: 2N7002, Package_TO_SOT_SMD:SOT-23
- removed R12: 100 Ohm, Resistor_SMD:R_0402_1005Metric
- removed R13: 10 kOhm, Resistor_SMD:R_0402_1005Metric
- removed R14: 100 kOhm, Resistor_SMD:R_0402_1005Metric
- added F1: 500mA, Fuse:Fuse_0603_1608Metric, B.Cu at (87.8, 109.9)
- added L1: BLM15PX121SN1D, Inductor_SMD:L_0402_1005Metric, B.Cu at (87.8, 112.5)
- added R1: 5k1, Resistor_SMD:R_0402_1005Metric, B.Cu at (96.3, 102.3)
- added R2: 5k1, Resistor_SMD:R_0402_1005Metric, B.Cu at (96.3, 101.2)
- added U4: SRV05-4, PCM_marbastlib-various:SOT-23-6-routable, B.Cu at (90.8, 109.1)
- J1: value JST -> TYPE-C-31-M-12; footprint Connector_JST:JST_SH_SM04B-SRSS-TB_1x04-1MP_P1.00mm_Horizontal -> PCM_marbastlib-various:USB_C_Receptacle_HRO_TYPE-C-31-M-12
- LED1, RST1: moved to F.Cu
- moved C1 170.7 mm to (89.0, 112.5), turned to 90 degrees
- moved U2 150.7 mm to (127.4, 135.9), turned to 0 degrees
- moved J2 143.8 mm to (111.2, 136.5), turned to -90 degrees
- moved R3 139.8 mm to (124.2, 136.9)
- moved R5 137.2 mm to (130.7, 136.9), turned to 0 degrees
- moved R4 137.0 mm to (127.7, 139.0), turned to -90 degrees
- moved R6 135.7 mm to (126.1, 138.5)
- moved U1 130.9 mm to (122.7, 139.1), turned to -90 degrees
- moved C6 130.5 mm to (122.2, 136.9)
- moved C8 129.0 mm to (123.9, 135.4), turned to 90 degrees
- moved C5 128.8 mm to (130.2, 135.4), turned to 90 degrees
- moved C7 128.8 mm to (122.7, 135.4), turned to 90 degrees
- moved C4 126.7 mm to (131.3, 135.4), turned to 90 degrees
- moved C3 125.2 mm to (129.2, 138.5), turned to 0 degrees
- moved C2 123.4 mm to (129.2, 139.6), turned to 0 degrees
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Connections:
- D46 pad 2: Net-(D46-A) -> wk3
- D47 pad 2: Net-(D47-A) -> wk2
- D48 pad 2: Net-(D48-A) -> wk1
- S46 pad 2: Net-(D46-A) -> wk3
- S47 pad 2: Net-(D47-A) -> wk2
- S48 pad 2: Net-(D48-A) -> wk1
- U2 pad 15: SYSOFF -> GND
- U3 pad 10: c11 -> unconnected-(U3-P0.30/AIN6-Pad10)
- U3 pad 12: r0 -> row1
- U3 pad 14: r1 -> row0
- U3 pad 16: r2 -> unconnected-(U3-P0.08-Pad16)
- U3 pad 2: unconnected-(U3-P1.10-Pad2) -> col1
- U3 pad 28: c03 -> col5
- U3 pad 3: c06 -> col3
- U3 pad 30: r3 -> col7
- U3 pad 32: c04 -> col9
- U3 pad 33: c05 -> row4
- U3 pad 34: c01 -> col8
- U3 pad 35: unconnected-(U3-P0.24-Pad35) -> col6
- U3 pad 36: LED_G -> col2
- U3 pad 38: LED_B -> col0
- U3 pad 4: c07 -> LED_G
- U3 pad 40: unconnected-(U3-P1.04-Pad40) -> col10
- U3 pad 41: c00 -> col11
- U3 pad 42: unconnected-(U3-P1.06-Pad42) -> col12
- U3 pad 43: c02 -> col13
- U3 pad 6: unconnected-(U3-P1.13-Pad6) -> LED_B
- U3 pad 7: c08 -> row2
- U3 pad 8: c09 -> row3
- U3 pad 9: c10 -> col4
Routing:
- net row2: track 0.00 -> 311.4 mm, vias 0 -> 4
- net row3: track 0.00 -> 311.1 mm, vias 0 -> 4
- net row0: track 0.00 -> 287.6 mm, vias 0 -> 2
- net row1: track 0.00 -> 284.9 mm, vias 0 -> 4
- net row4: track 0.00 -> 266.5 mm
- net col13: track 0.00 -> 261.7 mm
- net col12: track 0.00 -> 231.5 mm
- net col11: track 0.00 -> 211.8 mm
- net col10: track 0.00 -> 189.8 mm
- net col0: track 0.00 -> 188.4 mm
- net col9: track 0.00 -> 158.1 mm
- net col8: track 0.00 -> 157.3 mm
- net col1: track 0.00 -> 152.8 mm, vias 0 -> 1
- net col2: track 0.00 -> 151.6 mm
- net D+: track 0.00 -> 150.6 mm, vias 0 -> 2
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Other:
- board text added: "1t: reset 2t: bootloader"
- board text added: "R: Charging G: Bootloader/ FW controlled B: FW controlled"
