File: Hotp4ck60_rev.B/Hotpacky60_Matrix.kicad_sch (KiCad schematic)
At the start: 127 parts

Commit message: Change to daugtherboard
Parts:
- renumbered D62 to D57, D57 to D58, D58 to D59, D59 to D60, D60 to D61, D61 to D62, S62 to S?, S1 to S?, S2 to S?, S5 to S?, S58 to S?, S36 to S?, S60 to S?

Commit message: place parts and trace connect
Connections:
- net wk3: now reaches D46.2 (A), S?.2
- net wk1: now reaches D48.2 (A), S?.2
- net wk2: now reaches D47.2 (A), S?.2
Changed lines of the file:
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@@
 	(wire
 		(pts
-			(xy 22.86 90.17) (xy 27.94 90.17)
+			(xy 21.59 90.17) (xy 27.94 90.17)
 		)
 		(stroke
@@
 		)
 	)
+	(global_label "wk3"
+		(shape output)
+		(at 110.49 82.55 180)
+		(effects
+			(font
+				(size 1.27 1.27)
+			)
+			(justify right)
+		)
+		(property "Intersheetrefs" "${INTERSHEET_REFS}"
+			(at 88.9 -129.54 0)
+			(effects
+				(font
+					(size 1.27 1.27)
+				)
+				(hide yes)
+			)
+		)
+	)
 	(global_label "col11"
 		(shape input)
@@
 	(global_label "row4"
 		(shape output)
-		(at 22.86 90.17 180)
+		(at 21.59 90.17 180)
 		(effects
 			(font
@@
 		)
 		(property "Intersheetrefs" "${INTERSHEET_REFS}"
-			(at 1.27 -142.24 0)
+			(at 0 -142.24 0)
 			(effects
 				(font
@@
 			(effects
 				(font
+					(size 1.27 1.27)
+				)
+				(hide yes)
+			)
+		)
+	)
+	(global_label "wk2"
+		(shape output)
+		(at 127 82.55 180)
+		(effects
+			(font
+				(size 1.27 1.27)
+			)
+			(justify right)
+		)
+		(property "Intersheetrefs" "${INTERSHEET_REFS}"
+			(at 105.41 -109.22 0)
+			(effects
+				(font
+					(size 1.27 1.27)
+				)
+				(hide yes)
+			)
+		)
+	)
+	(global_label "wk1"
+		(shape output)
+		(at 143.51 82.55 180)
+		(effects
+			(font
+				(size 1.27 1.27)
+			)
+			(justify right)
+		)
+		(property "Intersheetrefs" "${INTERSHEET_REFS}"
+			(at 121.92 -88.9 0)
+			(effects
+				(font
