File: Hotp4ck60_rev.C/Hotp4ck60.kicad_pcb (KiCad board)
At the start: 2 copper layers, 284.7 x 94.2 mm, 169 parts, among them J1 Conn_01x04, J2 Conn_01x02_MountingPin, U1 MAX17048, U2 BQ24075, U3 nRF52840_E73-2G4M08S1C, Y1 32.768 KHz

Commit message: rev.c 핀, 트레이스 수정
Parts:
- removed L1: BLM15PX121SN1D, Inductor_SMD:L_0402_1005Metric
- R4: value 47k -> 15k
- R6: value 2k2 -> 910
- moved LED1 138.0 mm to (231.7, 184.2), turned to 90 degrees
- moved R11 136.5 mm to (229.5, 182.6), turned to 180 degrees
- moved R10 135.2 mm to (229.4, 184.2), turned to 180 degrees
- moved R9 134.2 mm to (229.4, 185.7), turned to 180 degrees
- moved J2 33.0 mm to (144.4, 135.2)
- moved D1 22.2 mm to (89.0, 110.3)
- moved J1 19.8 mm to (119.0, 116.5)
- moved D47 15.9 mm to (192.0, 158.0)
- moved D46 14.4 mm to (189.0, 158.0)
- moved F1 11.1 mm to (167.5, 139.9), turned to 180 degrees
- moved C1 10.9 mm to (170.1, 139.6), turned to 0 degrees
- moved D29 7.69 mm to (96.1, 148.4)
- moved J3 1.96 mm to (232.5, 176.0), turned to -90 degrees
- moved U1 0.22 mm to (163.9, 139.1)
- moved RST1 0.21 mm to (221.2, 182.3), turned to -90 degrees
Connections:
- F1 pad 1: Net-(F1-Pad1) -> +5V
- U3 pad 1: unconnected-(U3-P1.11-Pad1) -> col0
- U3 pad 12: row1 -> unconnected-(U3-P0.26-Pad12)
- U3 pad 14: row0 -> col7
- U3 pad 2: col1 -> col2
- U3 pad 20: unconnected-(U3-P0.12-Pad20) -> row1
- U3 pad 22: wk -> row0
- U3 pad 28: col7 -> row3
- U3 pad 30: col9 -> row2
- U3 pad 32: row3 -> col9
- U3 pad 34: col8 -> LED_G
- U3 pad 35: LED_G -> col10
- U3 pad 36: col2 -> LED_B
- U3 pad 38: col0 -> col8
- U3 pad 40: col10 -> col1
- U3 pad 6: LED_B -> col4
- U3 pad 7: col4 -> col5
- U3 pad 8: row2 -> unconnected-(U3-P0.29/AIN5-Pad8)
- U3 pad 9: col5 -> unconnected-(U3-P0.31/AIN7-Pad9)
Routing:
- net LED_G: track 190.9 -> 8.85 mm, vias 2 -> 0
- net LED_B: track 176.7 -> 9.50 mm, vias 2 -> 0
- net VDD: track 177.0 -> 35.4 mm, vias 2 -> 1
- net +BATT: track 72.0 -> 30.5 mm, vias 3 -> 1
- net D+: track 136.5 -> 171.6 mm, vias 2 -> 4
- net D-: track 136.4 -> 171.2 mm, vias 2 -> 4
- net row0: track 286.2 -> 314.0 mm
- net row3: track 301.1 -> 273.5 mm, vias 3 -> 1
- net VBUS: track 42.2 -> 69.3 mm, vias 2 -> 4
- net ~{CHG}: track 91.4 -> 116.2 mm
- net row1: track 355.8 -> 331.2 mm, vias 3 -> 2
- net Net-(D1-A): track 34.4 -> 10.7 mm
- net +5V: track 115.4 -> 96.7 mm, vias 3 -> 4
- net SWDCLK: track 9.58 -> 23.1 mm
- net col2: track 190.8 -> 178.1 mm
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Other:
- board text added: "3V3"
- board text added: "CLK"
- board text added: "IO"
- board text added: "R: G: B/L B:"
- board text added: "⏚"
- board text added: ""
- board text added: ""
- board text removed: "R: Charging G: Bootloader/ FW controlled B: FW controlled"

Commit message: README 수정
Parts:
- turned J2 to 90 degrees
Routing:
- net +BATT: track 30.5 -> 25.2 mm
Other:
- board text added: "+ POS RED"
- board text added: "- NEG BLK"

Commit message: LED 핀 수정
Parts:
- J1: value Conn_01x04 -> Conn_01x04_MountingPin
- J3: moved to F.Cu
- LED1: value IND -> LED_RAGB
- RST1: footprint PCM_marbastlib-various:SW_T1A2QR -> Button_Switch_SMD:SW_Push_1P1T_XKB_TS-1187A
- moved D46 16.0 mm to (173.0, 158.0)
- moved D47 15.9 mm to (207.9, 158.0)
- moved J3 6.49 mm to (233.1, 169.5), turned to 0 degrees
- moved R11 3.10 mm to (229.4, 185.7)
- moved R9 3.10 mm to (229.4, 182.6)
- moved RST1 2.04 mm to (220.3, 184.2)
- moved C10 1.98 mm to (225.6, 177.4), turned to -90 degrees
Connections:
- J1 pad MP: (no net) -> GND
- LED1 pad 1: VDD -> Net-(LED1-RK)
- LED1 pad 2: Net-(LED1-BK) -> VDD
- LED1 pad 4: Net-(LED1-RK) -> Net-(LED1-BK)
- U3 pad 34: LED_G -> LED_B
- U3 pad 36: LED_B -> LED_G
Routing:
- net D+: track 171.6 -> 154.5 mm
- net D-: track 171.2 -> 155.2 mm
- net ~{CHG}: track 116.2 -> 107.9 mm, vias 4 -> 6
- net SWDCLK: track 23.1 -> 17.5 mm
- net Net-(D47-A): track 11.0 -> 5.79 mm
- net Net-(D46-A): track 5.90 -> 11.0 mm
- net RST: track 8.56 -> 13.4 mm
- net row0: track 314.0 -> 309.3 mm
- net col5: track 115.9 -> 120.0 mm
- net col9: track 110.6 -> 114.4 mm
- net col7: track 80.4 -> 84.1 mm
- net col12: track 184.5 -> 187.9 mm
- net col1: track 209.4 -> 212.7 mm
- net col6: track 109.7 -> 113.1 mm
- net col10: track 135.9 -> 139.2 mm
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
Commit message: rev.C neocore
Parts:
- removed RST1: RST, Button_Switch_SMD:SW_Push_1P1T_XKB_TS-1187A
- removed the S1 at (81.0, 108.0)
- removed the S55 at (107.2, 184.2)
- removed the S60 at (273.8, 184.2)
- added D53: 1N4148WS, Diode_SMD:D_SOD-323, B.Cu at (266.6, 83.4)
- added S43: 1.00u, Switch_Keyboard_Cherry_MX:SW_Cherry_MX_PCB_1.00u, F.Cu at (83.3, 90.5)
- added S53: 1.75u, Switch_Keyboard_Cherry_MX:SW_Cherry_MX_PCB_1.75u, F.Cu at (281.0, 90.5)
- added S54_1: 1.00u, Switch_Keyboard_Cherry_MX:SW_Cherry_MX_PCB_1.00u, F.Cu at (307.2, 90.5)
- added S58: 1.25u, Switch_Keyboard_Cherry_MX:SW_Cherry_MX_PCB_1.25u, F.Cu at (114.3, 109.5)
- added S64: 1.25u, Switch_Keyboard_Cherry_MX:SW_Cherry_MX_PCB_1.25u, F.Cu at (304.8, 109.5)
- added SW1: SW_DIP_x01, hotp4ck:SW_DIP_HOTP4CK, F.Cu at (59.6, 71.5)
- H4: moved to B.Cu
- H8: value MountingHole -> Mounting_Keyboard_Stabilizer:6.25u; footprint amtra5_outline:Hotp4ckOutline -> hotp4ck:Neo60
- J1: value Conn_01x04_MountingPin -> Conn_01x05_Pin; footprint Connector_JST:JST_SH_SM04B-SRSS-TB_1x04-1MP_P1.00mm_Horizontal -> Connector_PinHeader_2.54mm:PinHeader_1x05_P2.54mm_Vertical; moved to F.Cu
- J2: value Conn_01x02_MountingPin -> Conn_01x05_Socket; footprint Connector_Molex:Molex_PicoBlade_53261-0271_1x02-1MP_P1.25mm_Horizontal -> Connector_PinSocket_2.54mm:PinSocket_1x05_P2.54mm_Vertical; moved to F.Cu
- J3: value ~ -> TC2030_SWD; footprint Connector_PinSocket_2.54mm:PinSocket_1x04_P2.54mm_Vertical -> PCM_marbastlib-various:CON_TC2030_outlined; moved to B.Cu
- LED1: value LED_RAGB -> LED_ABGR
- moved R11 215.1 mm to (44.4, 76.0)
- moved LED1 213.2 mm to (47.6, 76.5), turned to 180 degrees
- moved R10 207.6 mm to (50.9, 78.1), turned to 0 degrees
- moved R9 207.4 mm to (50.9, 77.1), turned to 0 degrees
- moved S1 155.9 mm to (40.5, 33.3)
- moved H2 119.0 mm to (297.7, 33.3), turned to 0 degrees
- moved D34 106.1 mm to (142.1, 73.8)
- moved S56 98.5 mm to (66.7, 109.5)
- moved S57 98.5 mm to (90.5, 109.5)
- moved S61 98.5 mm to (233.4, 109.5)
- moved S62 98.5 mm to (257.2, 109.5)
- moved S63 98.5 mm to (281.0, 109.5)
- moved D21 93.7 mm to (156.1, 54.8)
- moved D36 93.6 mm to (180.1, 73.8)
- moved J1 88.8 mm to (168.8, 42.9), turned to 90 degrees
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- renumbered D53 to D54, D54 to D55, D55 to D56, D56 to D57, D57 to D58, D58 to D59, D63 to D60, D59 to D61, D60 to D62, D61 to D63, D62 to D64, L2 to L1, S43 to S1, S53 to S54, S54 to S55, S58 to S59, S64 to S59_1, S59 to S60, U3 to U1, U1 to U3
Connections:
- C11 pad 1: +VSW -> +VDDH
- D56 pad 2: Net-(D55-A) (its old number) -> Net-(D56-A)
- D57 pad 2: Net-(D56-A) -> Net-(D57-A)
- D58 pad 2: Net-(D57-A) -> Net-(D58-A)
- D61 pad 2: Net-(D59-A) (its old number) -> Net-(D61-A)
- D62 pad 2: Net-(D60-A) (its old number) -> Net-(D62-A)
- D63 pad 2: Net-(D61-A) -> Net-(D63-A)
- D64 pad 2: Net-(D62-A) -> Net-(D64-A)
- J2 pad 1: +BATT -> VDD
- J2 pad 2: GND -> SWDIO
- J3 pad 3: SWDCLK -> RST
- J3 pad 4: GND -> SWDCLK
- LED1 pad 1: Net-(LED1-RK) -> VDD
- LED1 pad 2: VDD -> Net-(LED1-BK)
- LED1 pad 4: Net-(LED1-BK) -> Net-(LED1-RK)
- S1 pad 1: col2 -> col0
- S1 pad 2: Net-(D43-A) -> Net-(D1-A)
- S56 pad 1: col2 -> col1
- S57 pad 1: col3 -> col2
- S61 pad 1: col11 -> col10
- S61 pad 2: Net-(D60-A) (its old number) -> Net-(D61-A)
- S62 pad 1: col12 -> col11
- S62 pad 2: Net-(D61-A) -> Net-(D62-A)
- S63 pad 1: col13 -> col12
- S63 pad 2: Net-(D62-A) -> Net-(D63-A)
- U1 pad 10: unconnected-(U3-P0.30/AIN6-Pad10) -> LED_G
- U1 pad 12: unconnected-(U3-P0.26-Pad12) -> LED_B
- U1 pad 2: col2 -> col1
- U1 pad 20: row1 -> row2
- U1 pad 22: row0 -> row3
- U1 pad 23: +VSW -> +VDDH
- U1 pad 28: row3 -> row1
- U1 pad 30: row2 -> unconnected-(U1-P0.17-Pad30)
- U1 pad 32: col9 -> row0
- U1 pad 33: row4 -> unconnected-(U1-P0.13-Pad33)
- U1 pad 34: LED_B -> col9
- U1 pad 35: col10 -> row4
- U1 pad 36: LED_G -> col8
- U1 pad 38: col8 -> col2
- U1 pad 40: col1 -> col10
Routing:
- net +VDDH: track 0.00 -> 137.6 mm, vias 0 -> 1
- net VDD: track 36.4 -> 172.1 mm, vias 1 -> 2
- net LED_B: track 8.28 -> 142.6 mm
- net LED_G: track 8.63 -> 140.0 mm
- net D-: track 155.2 -> 76.1 mm, vias 4 -> 3
- net D+: track 154.5 -> 76.9 mm, vias 4 -> 3
- net +BATT: track 25.2 -> 81.0 mm, vias 1 -> 2
- net RST: track 13.4 -> 38.1 mm, vias 1 -> 2
- net Net-(D53-A): track 0.00 -> 17.4 mm
- net row3: track 273.5 -> 257.1 mm, vias 1 -> 2
- net row2: track 282.8 -> 269.0 mm, vias 2 -> 4
- net +5V: track 97.0 -> 110.6 mm
- net Net-(D34-A): track 29.1 -> 15.7 mm
- net Net-(D64-A): track 0.00 -> 13.3 mm
- net Net-(D54-A): track 5.88 -> 17.5 mm
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Other:
- outline, holes or cut-outs redrawn
- board text added: "+"
- board text added: "-"
- board text added: "R: G: B:"
- board text added: "RST"
- board text added: ""
- board text added: ""
- board text added: ""
- board text added: ""
- board text removed: "+ POS RED"
- board text removed: "- NEG BLK"
- board text removed: "R: G: B/L B:"
- board text removed: ""
- board text removed: ""
